Commit message: model done, working on auto connection method

File: src/amr_description/urdf/single_shelf.urdf.xacro (robot description, xacro)
@@ -19,5 +19,5 @@
 <xacro:property name="leg_radius" value="0.025"/>
 <xacro:property name="leg_length" value="0.32"/>
-<xacro:property name="leg_mass" value=".5"/>
+<xacro:property name="leg_mass" value="1"/>
 <!-- #####  leg macro  ##### -->
 <xacro:macro name="leg" params= "prefix suffix X1 X2 Y1 Y2">
@@ -29,5 +29,5 @@
   </joint>
   <link name= "${prefix}_${suffix}_leg">
-<!--
+    <!--
     <visual>
       <origin rpy= "0 0 0" xyz= "0 0 0"/>
@@ -37,5 +37,5 @@
       <material name= "light_black"/>
     </visual>
--->
+-->`
     <collision>
       <origin rpy= "0 0 0" xyz= "0 0 0"/>
@@ -47,8 +47,10 @@
   </link>
   <gazebo reference ="${prefix}_${suffix}_leg">
-    <mu1 value=".02"/>
-    <mu2 value=".02"/>
+    <mu1 value=".005"/>
+    <mu2 value=".005"/>
     <kp value="10000000.0"/>
-    <kd value= "1.0"/>
+    <kd value= "10.0"/>
+    <maxVel>0.</maxVel>
+    <minDepth>0.001</minDepth>
   </gazebo>
 </xacro:macro>
@@ -68,5 +70,5 @@
      </collision>
      <inertial>
-         <mass value="50.0"/>
+         <mass value="1.0"/>
               <inertia ixx="1.3542" ixy="0.0"
                        iyy="1.3542" iyz="0.0"
@@ -92,12 +94,19 @@
       <origin xyz="0.0 0 0.0" rpy="${PI} 0 ${PI/2}"/>
       <geometry>
+        <!--
         <mesh filename="package://amr_description/meshes/B_bot.stl" scale="0.01 0.01 0.01"/>
+-->
+        <mesh filename="package://amr_description/meshes/B_bot_shrink10mm.stl" scale="0.01 0.01 0.01"/>
       </geometry>
       <material name="light_black"/>
     </visual>
     <collision>
+      <max_contacts>1</max_contacts>
       <origin xyz="0.0 0 0.0" rpy="${PI} 0 ${PI/2}"/>
       <geometry>
+        <!--
         <mesh filename="package://amr_description/meshes/B_bot.stl" scale="0.01 0.01 0.01"/>
+-->
+        <mesh filename="package://amr_description/meshes/B_bot_shrink10mm.stl" scale="0.01 0.01 0.01"/>
       </geometry>
     </collision>
@@ -111,4 +120,10 @@
   </link>
   <gazebo reference="B_bot">
+      <mu1>0</mu1>
+      <mu2>0</mu2>
+      <kp>1000000</kp>
+      <kd>10</kd>
+      <maxVel>0.</maxVel>
+      <minDepth>0.001</minDepth>
       <material>Gazebo/Wood</material>
   </gazebo>

File: src/amr_description/urdf/solamr.gazebo.xacro (robot description, xacro)
@@ -9,7 +9,19 @@
   <gazebo reference="A2_top">
       <material>Gazebo/PointCloud</material>
+      <mu1>0</mu1>
+      <mu2>0</mu2>
+      <kp>1000000</kp>
+      <kd>10</kd>
+      <maxVel>0.</maxVel>
+      <minDepth>0.001</minDepth>
   </gazebo>
   <gazebo reference="blocker">
       <material>Gazebo/OrangeTransparentOverlay</material>
+      <mu1>0</mu1>
+      <mu2>0</mu2>
+      <kp>1000000</kp>
+      <kd>10</kd>
+      <maxVel>0.</maxVel>
+      <minDepth>0.001</minDepth>
   </gazebo>
   <gazebo reference="wheel_left_link">
@@ -33,4 +45,14 @@
     <material>Gazebo/FlatBlack</material>
   </gazebo>
+  <!--
+  <gazebo>
+    <plugin name="joint_state_publisher" filename="libgazebo_ros_joint_state_publisher.so">
+      <robotNamespace>$(arg robotName)</robotNamespace>
+      <jointName>rear_right_wheel_joint, rear_left_wheel_joint, front_right_wheel_joint, front_left_wheel_joint, front_right_steer_joint, front_left_steer_joint, steering_joint</jointName>
+      <updateRate>100.0</updateRate>
+      <alwaysOn>true</alwaysOn>
+    </plugin>
+  </gazebo>
+-->
   <gazebo>
     <plugin name="solamr_controller" filename="libgazebo_ros_diff_drive.so">
@@ -51,5 +73,5 @@
       <wheelDiameter>0.066</wheelDiameter>
       <wheelAcceleration>1</wheelAcceleration>
-      <wheelTorque>20</wheelTorque>
+      <wheelTorque>50</wheelTorque>
       <rosDebugLevel>na</rosDebugLevel>
     </plugin>
@@ -57,5 +79,5 @@
   <gazebo reference="scan_front">
     <material>Gazebo/FlatBlack</material>
-    <sensor type="ray" name="lds_lfcd_sensor">
+    <sensor type="ray" name="scan_front">
       <pose>0 0 0 0 0 0</pose>
       <visualize>$(arg laser_visual)</visualize>
@@ -78,5 +100,5 @@
           <type>gaussian</type>
           <mean>0.0</mean>
-          <stddev>0.01</stddev>
+          <stddev>0.0</stddev>
         </noise>
       </ray>
@@ -89,5 +111,5 @@
   <gazebo reference="scan_rear">
     <material>Gazebo/Blue</material>
-    <sensor type="ray" name="lds_lfcd_sensor">
+    <sensor type="ray" name="scan_rear">
       <pose>0 0 0 0 0 0</pose>
       <visualize>$(arg laser_visual)</visualize>
@@ -155,4 +177,5 @@
     </plugin>
   </gazebo>
+-->
   <gazebo reference="camera_rgb_frame">
     <sensor type="depth" name="realsense_R200">
@@ -198,4 +221,3 @@
     </sensor>
   </gazebo>
--->
 </robot>

File: src/amr_description/urdf/solamr.urdf.xacro (robot description, xacro)
@@ -3,4 +3,8 @@
   <xacro:include filename="$(find amr_description)/urdf/common_properties.xacro"/>
   <xacro:include filename="$(find amr_description)/urdf/solamr.gazebo.xacro"/>
+  <xacro:property name="r200_cam_rgb_px" value="0.005"/>
+  <xacro:property name="r200_cam_rgb_py" value="0.018"/>
+  <xacro:property name="r200_cam_rgb_pz" value="0.013"/>
+  <xacro:property name="r200_cam_depth_offset" value="0.01"/>
     <!-- #### constants #### -->
     <xacro:property name="deg_to_rad" value="0.017453"/>
@@ -32,14 +36,8 @@
       <link name= "${prefix}_${suffix}_caster">
         <visual>
-          <origin rpy= "${PI/2} 0 0" xyz= "0 0 0"/>
-          <geometry>
-            <cylinder length="${caster_length}" radius= "${caster_radius}"/>
-          </geometry>
-            <!--
           <origin rpy= "${PI/2} 0 0" xyz= "0 0 -0.025"/>
           <geometry>
             <mesh filename="package://amr_description/meshes/caster.stl" scale="0.0002 0.0002 0.0002"/>
           </geometry>
--->
           <material name= "grey"/>
         </visual>
@@ -91,31 +89,4 @@
     </inertial>
   </link>
-  <joint name="A2_top_joint" type="fixed">
-    <parent link="chassis"/>
-    <child link="A2_top" />
-    <origin xyz="0 0 0.18" rpy="0 0 0"/>
-  </joint>
-  <link name="A2_top">
-    <visual>
-      <origin xyz="0.0 0 0.0" rpy="0 0 -${PI/2}"/>
-      <geometry>
-        <mesh filename="package://amr_description/meshes/A2_top.stl" scale="0.01 0.01 0.01"/>
-      </geometry>
-      <material name="light_black"/>
-    </visual>
-    <collision>
-      <origin xyz="0.0 0 0.0" rpy="0 0 -${PI/2}"/>
-      <geometry>
-        <mesh filename="package://amr_description/meshes/A2_top.stl" scale="0.01 0.01 0.01"/>
-      </geometry>
-    </collision>
-    <inertial>
-      <origin xyz="0 0 0" rpy="0 0 0"/>
-      <mass value="1.5"/>
-      <inertia ixx="2.15625e-02" ixy="0" ixz="0"
-               iyy="2.15625e-02" iyz="0"
-               izz="2.25e-02" />
-    </inertial>
-  </link>
   <joint name="wheel_left_joint" type="continuous">
     <parent link="chassis"/>
@@ -245,4 +216,38 @@
 <!-- #####  A2 PART ##### -->
 <!-- #####   BEGIN  ##### -->
+  <joint name="A2_top_joint" type="fixed">
+    <parent link="chassis"/>
+    <child link="A2_top" />
+    <origin xyz="0 0 0.18" rpy="0 0 0"/>
+  </joint>
+  <link name="A2_top">
+    <visual>
+      <origin xyz="0.0 0 0.0" rpy="0 0 -${PI/2}"/>
+      <geometry>
+        <mesh filename="package://amr_description/meshes/A2_top_H.stl" scale="0.01 0.01 0.01"/>
+        <!--
+        <mesh filename="package://amr_description/meshes/A2_top_extr10mm_H.stl" scale="0.01 0.01 0.01"/>
+-->
+      </geometry>
+      <material name="light_black"/>
+    </visual>
+    <collision>
+      <max_contacts>1</max_contacts>
+      <origin xyz="0.0 0 0.0" rpy="0 0 -${PI/2}"/>
+      <geometry>
+        <mesh filename="package://amr_description/meshes/A2_top_H.stl" scale="0.01 0.01 0.01"/>
+        <!--
+        <mesh filename="package://amr_description/meshes/A2_top_extr10mm_H.stl" scale="0.01 0.01 0.01"/>
+-->
+      </geometry>
+    </collision>
+    <inertial>
+      <origin xyz="0 0 0" rpy="0 0 0"/>
+      <mass value="1.5"/>
+      <inertia ixx="2.15625e-02" ixy="0" ixz="0"
+               iyy="2.15625e-02" iyz="0"
+               izz="2.25e-02" />
+    </inertial>
+  </link>
   <transmission name="blocker_tran" type="SimpleTransmission">
     <type>transmission_interface/SimpleTransmission</type>
@@ -252,5 +257,5 @@
     <actuator name="blocker_motor">
       <hardwareInterface>EffortJointInterface</hardwareInterface>
-      <mechanicalReduction>1</mechanicalReduction>
+      <mechanicalReduction>500</mechanicalReduction>
     </actuator>
   </transmission>
@@ -263,5 +268,8 @@
   <link name="blocker">
     <visual>
+      <!--
       <origin xyz=".02 0 -0.0095" rpy="0 0 0"/>
+-->
+      <origin xyz=".02 0 -0.002" rpy="0 0 0"/>
       <geometry>
         <mesh filename="package://amr_description/meshes/blocker.stl" scale="0.0095 0.0095 0.0095"/>
@@ -270,5 +278,9 @@
     </visual>
     <collision>
+      <!--
       <origin xyz=".02 0 -0.0095" rpy="0 0 0"/>
+-->
+      <max_contacts>1</max_contacts>
+      <origin xyz=".02 0 -0.00" rpy="0 0 0"/>
       <geometry>
         <mesh filename="package://amr_description/meshes/blocker.stl" scale="0.0095 0.0095 0.0095"/>
@@ -293,7 +305,7 @@
 <!-- #####  A2 PART ##### -->
 <!-- #####    END   ##### -->
-<!--
+<!-- Begin of camera -->
   <joint name="camera_joint" type="fixed">
-    <origin xyz="0.064 -0.065 0.094" rpy="0 0 0"/>
+    <origin xyz="0.184 0 0.21" rpy="0 0 0"/>
     <parent link="chassis"/>
     <child link="camera_link"/>
@@ -306,4 +318,5 @@
       </geometry>
     </visual>
+    <!--
     <collision>
       <origin xyz="0.003 0.065 0.007" rpy="0 0 0"/>
@@ -312,4 +325,5 @@
       </geometry>
     </collision>
+-->
   </link>
   <joint name="camera_rgb_joint" type="fixed">
@@ -337,4 +351,4 @@
   </joint>
   <link name="camera_depth_optical_frame"/>
--->
+<!-- End of camera -->
 </robot>

Commit message: Tried LINE-MOD and find_object_2d, but both failed (due to short detection range. Now trying ArUco detecton (using ros aruco_detect pkg) which gives pose and orientation relative to camera_optical_frame. Successfully added a glowing ArUco in gazebo and tf_transform broadcaster is also written.)

File: src/amr_description/urdf/single_shelf.urdf.xacro (robot description, xacro)
@@ -12,4 +12,12 @@
      </inertial>
  </xacro:macro>
+<xacro:macro name="cuboid_inertia" params ="m w l h">
+    <inertial>
+        <mass value="${m}"/>
+        <inertia ixx="${m*(w*w+h*h)/12}" ixy="0.0" ixz="0.0"
+                 iyy="${m*(l*l+h*h)/12}" iyz= "0.0"
+                 izz="${m*(w*w+l*l)/12}"/>
+     </inertial>
+ </xacro:macro>
 <!-- #### body property #### -->
 <xacro:property name="body_length" value=".45"/>
@@ -21,13 +29,13 @@
 <xacro:property name="leg_mass" value="1"/>
 <!-- #####  leg macro  ##### -->
-<xacro:macro name="leg" params= "prefix suffix X1 X2 Y1 Y2">
+<xacro:macro name="leg" params= "prefix suffix X1 Y1">
   <joint name="${prefix}_${suffix}_leg_joint" type="fixed">
     <parent link= "body"/>
     <child link= "${prefix}_${suffix}_leg"/>
-    <origin xyz= "${(body_length/2)*X1 + (body_length/2)*X2} ${(body_width/2)*Y1 + (body_width/2)*Y2}  ${leg_length/2}" rpy="0 0 0"/>
+    <origin xyz= "${(body_length/2)*X1} ${(body_width/2)*Y1}  ${leg_length/2}" rpy="0 0 0"/>
     <dynamics damping="0.0" friction="0.0"/>
   </joint>
   <link name= "${prefix}_${suffix}_leg">
-    <!--
+    <!-- usefule to visualize when debugging
     <visual>
       <origin rpy= "0 0 0" xyz= "0 0 0"/>
@@ -37,5 +45,5 @@
       <material name= "light_black"/>
     </visual>
--->`
+    -->
     <collision>
       <origin rpy= "0 0 0" xyz= "0 0 0"/>
@@ -53,4 +61,38 @@
     <maxVel>0.</maxVel>
     <minDepth>0.001</minDepth>
+  </gazebo>
+</xacro:macro>
+<!-- ####  Aruco property #### -->
+<xacro:property name="aruco_width" value="0.4"/>
+<xacro:property name="aruco_length" value="0.4"/>
+<xacro:property name="aruco_height" value="0.01"/>
+<xacro:property name="aruco_z" value="1."/>
+<xacro:property name="aruco_mass" value="1"/>
+<!-- #####  Aruco macro  ##### -->
+    <!-- Aruco facing -->
+<xacro:macro name="aruco" params= "prefix X1 Y1 Yaw">
+  <joint name="${prefix}_joint" type="fixed">
+    <parent link= "body"/>
+    <child link= "${prefix}_aruco"/>
+    <origin xyz= "${(body_length/2)*X1} ${(body_width/2)*Y1} ${aruco_z}" rpy="${PI/2} 0 ${Yaw*PI/2}"/>
+    <dynamics damping="0.0" friction="0.0"/>
+  </joint>
+  <link name= "${prefix}_aruco">
+    <visual>
+      <origin rpy= "0 0 0" xyz= "0 0 0"/>
+      <geometry>
+          <box size="${aruco_length} ${aruco_width} ${aruco_height}"/>
+      </geometry>
+    </visual>
+    <collision>
+      <origin rpy= "0 0 0" xyz= "0 0 0"/>
+      <geometry>
+          <box size="${aruco_length} ${aruco_width} ${aruco_height}"/>
+      </geometry>
+    </collision>
+    <xacro:cuboid_inertia m="${aruco_mass}" w="${aruco_width}" l="${aruco_length}" h="${aruco_height}"/>
+  </link>
+  <gazebo reference="${prefix}_aruco">
+      <material>aruco/0</material>
   </gazebo>
 </xacro:macro>
@@ -80,8 +122,8 @@
   </gazebo>
 <!-- #### 4 legs #### -->
-  <xacro:leg prefix="right" suffix="front" X1="0" X2="1" Y1="-1" Y2="0" />
-  <xacro:leg prefix="right" suffix="back" X1="-1" X2="0" Y1="-1" Y2="0"/>
-  <xacro:leg prefix="left" suffix="front" X1="0" X2="1" Y1="0" Y2="1"/>
-  <xacro:leg prefix="left" suffix="back" X1="-1" X2="0" Y1="0" Y2="1"/>
+  <xacro:leg prefix="right" suffix="front" X1="1" Y1="-1"/>
+  <xacro:leg prefix="right" suffix="back" X1="-1" Y1="-1"/>
+  <xacro:leg prefix="left" suffix="front" X1="1" Y1="1"/>
+  <xacro:leg prefix="left" suffix="back" X1="-1" Y1="1"/>
 <!-- #### B bottom #### -->
   <joint name="B_bot_joint" type="fixed">
@@ -96,5 +138,5 @@
         <!--
         <mesh filename="package://amr_description/meshes/B_bot.stl" scale="0.01 0.01 0.01"/>
--->
+        -->
         <mesh filename="package://amr_description/meshes/B_bot_shrink10mm.stl" scale="0.01 0.01 0.01"/>
       </geometry>
@@ -107,5 +149,5 @@
         <!--
         <mesh filename="package://amr_description/meshes/B_bot.stl" scale="0.01 0.01 0.01"/>
--->
+        -->
         <mesh filename="package://amr_description/meshes/B_bot_shrink10mm.stl" scale="0.01 0.01 0.01"/>
       </geometry>
@@ -119,4 +161,9 @@
     </inertial>
   </link>
+  <!-- Aruco spawn -->
+  <xacro:aruco prefix="east" X1="0" Y1="-1" Yaw="0" />
+  <xacro:aruco prefix="west" X1="0" Y1="1" Yaw="0" />
+  <xacro:aruco prefix="north" X1="1" Y1="0" Yaw="1" />
+  <xacro:aruco prefix="south" X1="-1" Y1="0" Yaw="1" />
   <gazebo reference="B_bot">
       <mu1>0</mu1>

File: src/amr_description/urdf/solamr.gazebo.xacro (robot description, xacro)
@@ -185,11 +185,15 @@
           <horizontal_fov>1.3439</horizontal_fov>
           <image>
-              <width>1920</width>
-              <height>1080</height>
+              <!--
+              <width>1280</width>
+              <height>720</height>
+-->
+              <width>640</width>
+              <height>480</height>
               <format>R8G8B8</format>
           </image>
           <depth_camera></depth_camera>
           <clip>
-              <near>0.03</near>
+              <near>0.1</near>
               <far>100</far>
           </clip>

Commit message: ArUco on the shelft will be identified and saved in the dictionary. The rule for the ArUco ID should be documented and the last digit should be within 0, 1, 2, 3 which stand for the four sides of the shelft

File: src/amr_description/urdf/single_shelf.urdf.xacro (robot description, xacro)
@@ -64,11 +64,12 @@
 </xacro:macro>
 <!-- ####  Aruco property #### -->
-<xacro:property name="aruco_width" value="0.4"/>
-<xacro:property name="aruco_length" value="0.4"/>
+<xacro:property name="aruco_width" value="0.25"/>
+<xacro:property name="aruco_length" value="0.25"/>
 <xacro:property name="aruco_height" value="0.01"/>
 <xacro:property name="aruco_z" value="1."/>
 <xacro:property name="aruco_mass" value="1"/>
+<xacro:property name="edge_width" value="0.1"/>
 <!-- #####  Aruco macro  ##### -->
-    <!-- Aruco facing -->
+    <!-- Aruco facing four directions-->
 <xacro:macro name="aruco" params= "prefix X1 Y1 Yaw">
   <joint name="${prefix}_joint" type="fixed">
@@ -94,5 +95,30 @@
   </link>
   <gazebo reference="${prefix}_aruco">
-      <material>aruco/0</material>
+      <material>SOLab/aruco0</material>
+  </gazebo>
+    <!-- Back Board for white edges -->
+  <joint name="${prefix}_whiteboarder_joint" type="fixed">
+    <parent link= "body"/>
+    <child link= "${prefix}_aruco_whiteboarder"/>
+    <origin xyz= "${(body_length/2-aruco_height*1/3)*X1} ${(body_width/2-aruco_height*1/3)*Y1} ${aruco_z}" rpy="${PI/2} 0 ${Yaw*PI/2}"/>
+    <dynamics damping="0.0" friction="0.0"/>
+  </joint>
+  <link name= "${prefix}_aruco_whiteboarder">
+    <visual>
+      <origin rpy= "0 0 0" xyz= "0 0 0"/>
+      <geometry>
+          <box size="${aruco_length+edge_width} ${aruco_width+edge_width} ${aruco_height}"/>
+      </geometry>
+    </visual>
+    <collision>
+      <origin rpy= "0 0 0" xyz= "0 0 0"/>
+      <geometry>
+          <box size="${aruco_length+edge_width} ${aruco_width+edge_width} ${aruco_height}"/>
+      </geometry>
+    </collision>
+    <xacro:cuboid_inertia m="${aruco_mass}" w="${aruco_width+edge_width}" l="${aruco_length+edge_width}" h="${aruco_height}"/>
+  </link>
+  <gazebo reference="${prefix}_aruco_whiteboarder">
+      <material>SOLab/WhiteGlow</material>
   </gazebo>
 </xacro:macro>

Commit message: Done Tracking shelfts!

File: src/amr_description/urdf/single_shelf.urdf.xacro (robot description, xacro)
@@ -72,5 +72,5 @@
 <!-- #####  Aruco macro  ##### -->
     <!-- Aruco facing four directions-->
-<xacro:macro name="aruco" params= "prefix X1 Y1 Yaw">
+<xacro:macro name="aruco" params= "prefix X1 Y1 Yaw aruco_id">
   <joint name="${prefix}_joint" type="fixed">
     <parent link= "body"/>
@@ -95,5 +95,5 @@
   </link>
   <gazebo reference="${prefix}_aruco">
-      <material>SOLab/aruco0</material>
+      <material>SOLab/aruco${aruco_id}</material>
   </gazebo>
     <!-- Back Board for white edges -->
@@ -188,8 +188,8 @@
   </link>
   <!-- Aruco spawn -->
-  <xacro:aruco prefix="east" X1="0" Y1="-1" Yaw="0" />
-  <xacro:aruco prefix="west" X1="0" Y1="1" Yaw="0" />
-  <xacro:aruco prefix="north" X1="1" Y1="0" Yaw="1" />
-  <xacro:aruco prefix="south" X1="-1" Y1="0" Yaw="1" />
+  <xacro:aruco prefix="east" X1="0" Y1="-1" Yaw="0" aruco_id="203"/>
+  <xacro:aruco prefix="west" X1="0" Y1="1" Yaw="0"  aruco_id="201"/>
+  <xacro:aruco prefix="north" X1="1" Y1="0" Yaw="1" aruco_id="200"/>
+  <xacro:aruco prefix="south" X1="-1" Y1="0" Yaw="1" aruco_id="202"/>
   <gazebo reference="B_bot">
       <mu1>0</mu1>

File: src/amr_description/urdf/solamr.urdf.xacro (robot description, xacro)
@@ -307,5 +307,5 @@
 <!-- Begin of camera -->
   <joint name="camera_joint" type="fixed">
-    <origin xyz="0.184 0 0.21" rpy="0 0 0"/>
+    <origin xyz="0.33 0 0.161" rpy="0 0 0"/>
     <parent link="chassis"/>
     <child link="camera_link"/>
