Commit message: SOLAMR models are done : solamr, single_shelf, blocker. Control of SOLAMR and blocker are also done. Problem : shelf will jump around when SOLAMR is pushing/draging it.

File: src/amr_description/urdf/solamr.gazebo.xacro (robot description, xacro)
@@ -1,27 +1,33 @@
 <?xml version="1.0"?>
-<robot name="solamr" xmlns:xacro="http://ros.org/wiki/xacro">
+<robot name="$(arg robotName)" xmlns:xacro="http://ros.org/wiki/xacro">
   <xacro:arg name="laser_visual"  default="false"/>
   <xacro:arg name="camera_visual" default="false"/>
   <xacro:arg name="imu_visual"    default="false"/>
-  <gazebo reference="base_link">
-    <material>Gazebo/DarkGrey</material>
+  <gazebo reference="chassis">
+      <material>Gazebo/CeilingTiled</material>
+  </gazebo>
+  <gazebo reference="A2_top">
+      <material>Gazebo/PointCloud</material>
+  </gazebo>
+  <gazebo reference="blocker">
+      <material>Gazebo/OrangeTransparentOverlay</material>
   </gazebo>
   <gazebo reference="wheel_left_link">
-    <mu1>0.1</mu1>
-    <mu2>0.1</mu2>
-    <kp>500000.0</kp>
+    <mu1>20</mu1>
+    <mu2>20</mu2>
+    <kp>50000.0</kp>
     <kd>10.0</kd>
     <minDepth>0.001</minDepth>
-    <maxVel>0.1</maxVel>
+    <maxVel>3</maxVel>
     <fdir1>1 0 0</fdir1>
     <material>Gazebo/FlatBlack</material>
   </gazebo>
   <gazebo reference="wheel_right_link">
-    <mu1>0.1</mu1>
-    <mu2>0.1</mu2>
-    <kp>500000.0</kp>
+    <mu1>20</mu1>
+    <mu2>20</mu2>
+    <kp>50000.0</kp>
     <kd>10.0</kd>
     <minDepth>0.001</minDepth>
-    <maxVel>0.1</maxVel>
+    <maxVel>3</maxVel>
     <fdir1>1 0 0</fdir1>
     <material>Gazebo/FlatBlack</material>
@@ -42,30 +48,76 @@
       <leftJoint>wheel_left_joint</leftJoint>
       <rightJoint>wheel_right_joint</rightJoint>
-      <wheelSeparation>0.287</wheelSeparation>
+      <wheelSeparation>0.20</wheelSeparation>
       <wheelDiameter>0.066</wheelDiameter>
       <wheelAcceleration>1</wheelAcceleration>
-      <wheelTorque>10</wheelTorque>
+      <wheelTorque>20</wheelTorque>
       <rosDebugLevel>na</rosDebugLevel>
     </plugin>
   </gazebo>
+  <gazebo reference="scan_front">
+    <material>Gazebo/FlatBlack</material>
+    <sensor type="ray" name="lds_lfcd_sensor">
+      <pose>0 0 0 0 0 0</pose>
+      <visualize>$(arg laser_visual)</visualize>
+      <update_rate>5</update_rate>
+      <ray>
+        <scan>
+          <horizontal>
+            <samples>300</samples>
+            <resolution>1</resolution>
+            <min_angle>0.0</min_angle>
+            <max_angle>4.712</max_angle>
+          </horizontal>
+        </scan>
+        <range>
+          <min>0.120</min>
+          <max>3.5</max>
+          <resolution>0.015</resolution>
+        </range>
+        <noise>
+          <type>gaussian</type>
+          <mean>0.0</mean>
+          <stddev>0.01</stddev>
+        </noise>
+      </ray>
+      <plugin name="gazebo_ros_lds_lfcd_controller" filename="libgazebo_ros_laser.so">
+        <topicName>scan_front</topicName>
+        <frameName>scan_front</frameName>
+      </plugin>
+    </sensor>
+  </gazebo>
+  <gazebo reference="scan_rear">
+    <material>Gazebo/Blue</material>
+    <sensor type="ray" name="lds_lfcd_sensor">
+      <pose>0 0 0 0 0 0</pose>
+      <visualize>$(arg laser_visual)</visualize>
+      <update_rate>5</update_rate>
+      <ray>
+        <scan>
+          <horizontal>
+            <samples>300</samples>
+            <resolution>1</resolution>
+            <min_angle>0.0</min_angle>
+            <max_angle>4.712</max_angle>
+          </horizontal>
+        </scan>
+        <range>
+          <min>0.120</min>
+          <max>3.5</max>
+          <resolution>0.015</resolution>
+        </range>
+        <noise>
+          <type>gaussian</type>
+          <mean>0.0</mean>
+          <stddev>0.01</stddev>
+        </noise>
+      </ray>
+      <plugin name="gazebo_ros_lds_lfcd_controller" filename="libgazebo_ros_laser.so">
+        <topicName>scan_rear</topicName>
+        <frameName>scan_rear</frameName>
+      </plugin>
+    </sensor>
+  </gazebo>
 <!--
-  <gazebo reference="caster_back_right_link">
-    <mu1>0.1</mu1>
-    <mu2>0.1</mu2>
-    <kp>1000000.0</kp>
-    <kd>100.0</kd>
-    <minDepth>0.001</minDepth>
-    <maxVel>1.0</maxVel>
-    <material>Gazebo/FlatBlack</material>
-  </gazebo>
-  <gazebo reference="caster_back_left_link">
-    <mu1>0.1</mu1>
-    <mu2>0.1</mu2>
-    <kp>1000000.0</kp>
-    <kd>100.0</kd>
-    <minDepth>0.001</minDepth>
-    <maxVel>1.0</maxVel>
-    <material>Gazebo/FlatBlack</material>
-  </gazebo>
   <gazebo reference="imu_link">
     <sensor type="imu" name="imu">
@@ -102,36 +154,4 @@
       </imu>
     </plugin>
-  </gazebo>
-  <gazebo reference="base_scan">
-    <material>Gazebo/FlatBlack</material>
-    <sensor type="ray" name="lds_lfcd_sensor">
-      <pose>0 0 0 0 0 0</pose>
-      <visualize>$(arg laser_visual)</visualize>
-      <update_rate>5</update_rate>
-      <ray>
-        <scan>
-          <horizontal>
-            <samples>360</samples>
-            <resolution>1</resolution>
-            <min_angle>0.0</min_angle>
-            <max_angle>6.28319</max_angle>
-          </horizontal>
-        </scan>
-        <range>
-          <min>0.120</min>
-          <max>3.5</max>
-          <resolution>0.015</resolution>
-        </range>
-        <noise>
-          <type>gaussian</type>
-          <mean>0.0</mean>
-          <stddev>0.01</stddev>
-        </noise>
-      </ray>
-      <plugin name="gazebo_ros_lds_lfcd_controller" filename="libgazebo_ros_laser.so">
-        <topicName>scan</topicName>
-        <frameName>base_scan</frameName>
-      </plugin>
-    </sensor>
   </gazebo>
   <gazebo reference="camera_rgb_frame">

File: src/amr_description/urdf/solamr.urdf.xacro (robot description, xacro)
@@ -1,23 +1,77 @@
 <?xml version="1.0" ?>
-<robot name="solamr" xmlns:xacro="http://ros.org/wiki/xacro">
+<robot name="$(arg robotName)" xmlns:xacro="http://ros.org/wiki/xacro">
   <xacro:include filename="$(find amr_description)/urdf/common_properties.xacro"/>
   <xacro:include filename="$(find amr_description)/urdf/solamr.gazebo.xacro"/>
-<!-- Add some macro file and color properties which are not needed yet
-  <xacro:property name="r200_cam_rgb_px" value="0.005"/>
-  <xacro:property name="r200_cam_rgb_py" value="0.018"/>
-  <xacro:property name="r200_cam_rgb_pz" value="0.013"/>
-  <xacro:property name="r200_cam_depth_offset" value="0.01"/>
+    <!-- #### constants #### -->
+    <xacro:property name="deg_to_rad" value="0.017453"/>
+    <xacro:property name="PI" value="3.14"/>
+    <xacro:macro name="cylinder_inertia" params ="m r h">
+        <inertial>
+            <mass value="${m}"/>
+            <inertia ixx="${m*(3*r*r+h*h)/12}" ixy="0.0" ixz="0.0"
+                     iyy="${m*(3*r*r+h*h)/12}" iyz= "0.0"
+                     izz="${m*r*r/2}"/>
+         </inertial>
+     </xacro:macro>
+    <!-- #### chassis property #### -->
+    <xacro:property name="chassis_length" value=".65"/>
+    <xacro:property name="chassis_width" value=".3"/>
+    <xacro:property name="chassis_height" value="0.05"/>
+    <!-- ####  caster property #### -->
+    <xacro:property name="caster_radius" value="0.025"/>
+    <xacro:property name="caster_length" value="0.015"/>
+    <xacro:property name="caster_mass" value=".2"/>
+    <!-- #####  caster macro  ##### -->
+    <xacro:macro name="caster" params= "prefix suffix X1 X2 Y1 Y2">
+      <joint name="${prefix}_${suffix}_caster_joint" type="fixed">
+        <parent link= "chassis"/>
+        <child link= "${prefix}_${suffix}_caster"/>
+        <origin xyz= "${(chassis_length/2)*X1 + (chassis_length/2-.05)*X2} ${(chassis_width/2-0.02)*Y1 + (chassis_width/2)*Y2}  0.026" rpy="0 0 0"/>
+        <dynamics damping="0.0" friction="0.0"/>
+      </joint>
+      <link name= "${prefix}_${suffix}_caster">
+        <visual>
+          <origin rpy= "${PI/2} 0 0" xyz= "0 0 0"/>
+          <geometry>
+            <cylinder length="${caster_length}" radius= "${caster_radius}"/>
+          </geometry>
+            <!--
+          <origin rpy= "${PI/2} 0 0" xyz= "0 0 -0.025"/>
+          <geometry>
+            <mesh filename="package://amr_description/meshes/caster.stl" scale="0.0002 0.0002 0.0002"/>
+          </geometry>
 -->
+          <material name= "grey"/>
+        </visual>
+        <collision>
+          <origin rpy= "${PI/2} 0 0" xyz= "0 0 0"/>
+          <geometry>
+            <cylinder length="${caster_length}" radius= "${caster_radius}"/>
+          </geometry>
+        </collision>
+        <xacro:cylinder_inertia m="${caster_mass}" r="${caster_radius}" h="${caster_length}"/>
+      </link>
+      <gazebo reference ="${prefix}_${suffix}_caster">
+        <mu1 value="0.001"/>
+        <mu2 value="0.001"/>
+        <kp value="10000000.0"/>
+        <kd value= "1.0"/>
+        <material>Gazebo/WhiteGlow</material>
+      </gazebo>
+    </xacro:macro>
   <link name="base_footprint"/>
+<!-- #####   BEGIN  ##### -->
+<!-- #####  A1 PART ##### -->
+<!-- #####   BEGIN  ##### -->
   <joint name="base_joint" type="fixed">
     <parent link="base_footprint"/>
-    <child link="base_link" />
+    <child link="chassis" />
     <origin xyz="0 0 0.0" rpy="0 0 0"/>
   </joint>
-  <link name="base_link">
+  <link name="chassis">
     <visual>
       <origin xyz="0.0 0 0.075" rpy="0 0 0"/>
       <geometry>
-        <box size="0.30 0.30 0.05"/>
+        <box size="${chassis_length} ${chassis_width} ${chassis_height}"/>
       </geometry>
       <material name="light_black"/>
@@ -26,5 +80,32 @@
       <origin xyz="0.0 0 0.075" rpy="0 0 0"/>
       <geometry>
-        <box size="0.30 0.30 0.05"/>
+        <box size="${chassis_length} ${chassis_width} ${chassis_height}"/>
+      </geometry>
+    </collision>
+    <inertial>
+      <origin xyz="0 0 0" rpy="0 0 0"/>
+      <mass value="15"/>
+      <inertia ixx="1.15625e-01" ixy="0" ixz="0"
+               iyy="1.15625e-01" iyz="0"
+               izz="2.25e-01" />
+    </inertial>
+  </link>
+  <joint name="A2_top_joint" type="fixed">
+    <parent link="chassis"/>
+    <child link="A2_top" />
+    <origin xyz="0 0 0.18" rpy="0 0 0"/>
+  </joint>
+  <link name="A2_top">
+    <visual>
+      <origin xyz="0.0 0 0.0" rpy="0 0 -${PI/2}"/>
+      <geometry>
+        <mesh filename="package://amr_description/meshes/A2_top.stl" scale="0.01 0.01 0.01"/>
+      </geometry>
+      <material name="light_black"/>
+    </visual>
+    <collision>
+      <origin xyz="0.0 0 0.0" rpy="0 0 -${PI/2}"/>
+      <geometry>
+        <mesh filename="package://amr_description/meshes/A2_top.stl" scale="0.01 0.01 0.01"/>
       </geometry>
     </collision>
@@ -32,13 +113,13 @@
       <origin xyz="0 0 0" rpy="0 0 0"/>
       <mass value="1.5"/>
-      <inertia ixx="1.15625e-02" ixy="0" ixz="0"
-               iyy="1.15625e-02" iyz="0"
+      <inertia ixx="2.15625e-02" ixy="0" ixz="0"
+               iyy="2.15625e-02" iyz="0"
                izz="2.25e-02" />
     </inertial>
   </link>
   <joint name="wheel_left_joint" type="continuous">
-    <parent link="base_link"/>
+    <parent link="chassis"/>
     <child link="wheel_left_link"/>
-    <origin xyz="0.0 0.10 0.033" rpy="-1.57 0 0"/>
+    <origin xyz="0.0 ${chassis_width/2-0.05} 0.033" rpy="-1.57 0 0"/>
     <axis xyz="0 0 1"/>
   </joint>
@@ -66,7 +147,7 @@
   </link>
   <joint name="wheel_right_joint" type="continuous">
-    <parent link="base_link"/>
+    <parent link="chassis"/>
     <child link="wheel_right_link"/>
-    <origin xyz="0.0 -0.10 0.033" rpy="-1.57 0 0"/>
+    <origin xyz="0.0 -${chassis_width/2-0.05} 0.033" rpy="-1.57 0 0"/>
     <axis xyz="0 0 1"/>
   </joint>
@@ -93,76 +174,27 @@
       </inertial>
   </link>
-<!--
-  <joint name="caster_back_right_joint" type="fixed">
-    <parent link="base_link"/>
-    <child link="caster_back_right_link"/>
-    <origin xyz="-0.15 0.0 0.025" rpy="0 0 0"/>
-  </joint>
-  <link name="caster_back_right_link">
-    <visual>
-      <origin xyz="0 0.001 0" rpy="0 0 0"/>
-      <geometry>
-        <box size="0.030 0.009 0.050"/>
-      </geometry>
-    </visual>
-    <collision>
-      <origin xyz="0 0.001 0" rpy="0 0 0"/>
-      <geometry>
-        <box size="0.030 0.009 0.050"/>
-      </geometry>
-    </collision>
-    <inertial>
-      <origin xyz="0 0 0" />
-      <mass value="0.005" />
-      <inertia ixx="0.001" ixy="0.0" ixz="0.0"
-               iyy="0.001" iyz="0.0"
-               izz="0.001" />
-    </inertial>
-  </link>
-  <joint name="caster_back_left_joint" type="fixed">
-    <parent link="base_link"/>
-    <child link="caster_back_left_link"/>
-    <origin xyz="0.15 0.0 0.025" rpy="-1.57 0 0"/>
-  </joint>
-  <link name="caster_back_left_link">
-    <collision>
-      <origin xyz="0 0.001 0" rpy="0 0 0"/>
-      <geometry>
-        <box size="0.030 0.009 0.050"/>
-      </geometry>
-    </collision>
-    <inertial>
-      <origin xyz="0 0 0" />
-      <mass value="0.005" />
-      <inertia ixx="0.001" ixy="0.0" ixz="0.0"
-               iyy="0.001" iyz="0.0"
-               izz="0.001" />
-    </inertial>
-  </link>
--->
-<!--
-  <joint name="imu_joint" type="fixed">
-    <parent link="base_link"/>
-    <child link="imu_link"/>
-    <origin xyz="0.0 0 0.068" rpy="0 0 0"/>
-  </joint>
-  <link name="imu_link"/>
-  <joint name="scan_joint" type="fixed">
-    <parent link="base_link"/>
-    <child link="base_scan"/>
-    <origin xyz="-0.064 0 0.122" rpy="0 0 0"/>
-  </joint>
-  <link name="base_scan">
-    <visual>
-      <origin xyz="0 0 0" rpy="0 0 0"/>
-      <geometry>
-        <mesh filename="package://turtlebot3_description/meshes/sensors/lds.stl" scale="0.001 0.001 0.001"/>
-      </geometry>
-      <material name="dark"/>
-    </visual>
-    <collision>
-      <origin xyz="0.015 0 -0.0065" rpy="0 0 0"/>
-      <geometry>
-        <cylinder length="0.0315" radius="0.055"/>
+<!-- #### 4 casters #### -->
+  <xacro:caster prefix="right" suffix="front" X1="0" X2="1" Y1="-1" Y2="0" />
+  <xacro:caster prefix="right" suffix="back" X1="-1" X2="0" Y1="-1" Y2="0"/>
+  <xacro:caster prefix="left" suffix="front" X1="0" X2="1" Y1="0" Y2="1"/>
+  <xacro:caster prefix="left" suffix="back" X1="-1" X2="0" Y1="0" Y2="1"/>
+<!-- #### Sensors : Lidar #### -->
+  <joint name="scan_joint1" type="fixed">
+    <parent link="chassis"/>
+    <child link="scan_front"/>
+    <origin xyz="${chassis_length/2-0.03} ${chassis_width/2-0.03} 0.16" rpy="0 0 -${PI/2}"/>
+  </joint>
+  <link name="scan_front">
+    <visual>
+      <origin xyz="0 0 -.06" rpy="${PI/2} 0 0"/>
+      <geometry>
+        <mesh filename="package://amr_description/meshes/sensors/hokuyo_lidar.stl" scale="0.012 0.012 0.012"/>
+      </geometry>
+      <material name="black"/>
+    </visual>
+    <collision>
+      <origin xyz="0 0 -.03" rpy="0 0 0"/>
+      <geometry>
+        <cylinder length="0.08" radius="0.025"/>
       </geometry>
     </collision>
@@ -175,7 +207,94 @@
     </inertial>
   </link>
+  <joint name="scan_joint2" type="fixed">
+    <parent link="chassis"/>
+    <child link="scan_rear"/>
+    <origin xyz="-${chassis_length/2-0.03} -${chassis_width/2-0.03} 0.16" rpy="0 0 ${PI/2}"/>
+  </joint>
+  <link name="scan_rear">
+    <visual>
+      <origin xyz="0 0 -.06" rpy="${PI/2} 0 0"/>
+      <geometry>
+        <mesh filename="package://amr_description/meshes/sensors/hokuyo_lidar.stl" scale="0.012 0.012 0.012"/>
+      </geometry>
+      <material name="blue"/>
+    </visual>
+    <collision>
+      <origin xyz="0 0 -0.03" rpy="0 0 0"/>
+      <geometry>
+        <cylinder length="0.08" radius="0.025"/>
+      </geometry>
+    </collision>
+    <inertial>
+      <mass value="0.114" />
+      <origin xyz="0 0 0" />
+      <inertia ixx="0.001" ixy="0.0" ixz="0.0"
+               iyy="0.001" iyz="0.0"
+               izz="0.001" />
+    </inertial>
+  </link>
+<!-- #####    END   ##### -->
+<!-- #####  A1 PART ##### -->
+<!-- #####    END   ##### -->
+<gazebo>
+  <plugin name="gazebo_ros_control" filename="libgazebo_ros_control.so">
+    <robotSimType>gazebo_ros_control/DefaultRobotHWSim</robotSimType>
+  </plugin>
+</gazebo>
+<!-- #####   BEGIN  ##### -->
+<!-- #####  A2 PART ##### -->
+<!-- #####   BEGIN  ##### -->
+  <transmission name="blocker_tran" type="SimpleTransmission">
+    <type>transmission_interface/SimpleTransmission</type>
+    <joint name="blocker_joint">
+      <hardwareInterface>EffortJointInterface</hardwareInterface>
+    </joint>
+    <actuator name="blocker_motor">
+      <hardwareInterface>EffortJointInterface</hardwareInterface>
+      <mechanicalReduction>1</mechanicalReduction>
+    </actuator>
+  </transmission>
+  <joint name="blocker_joint" type="continuous">
+    <parent link="chassis"/>
+    <child link="blocker"/>
+    <origin xyz="0.083 0 .18" rpy="0 1.57 0"/>
+    <axis xyz="0 0 1"/>
+  </joint>
+  <link name="blocker">
+    <visual>
+      <origin xyz=".02 0 -0.0095" rpy="0 0 0"/>
+      <geometry>
+        <mesh filename="package://amr_description/meshes/blocker.stl" scale="0.0095 0.0095 0.0095"/>
+      </geometry>
+      <material name="orange"/>
+    </visual>
+    <collision>
+      <origin xyz=".02 0 -0.0095" rpy="0 0 0"/>
+      <geometry>
+        <mesh filename="package://amr_description/meshes/blocker.stl" scale="0.0095 0.0095 0.0095"/>
+      </geometry>
+    </collision>
+    <gazebo reference ="blocker">
+      <material>Gazebo/Orange</material>
+      <turnGravityOff>false</turnGravityOff>
+    </gazebo>
+    <inertial>
+      <origin xyz="0 0 0" rpy="0 0 0"/>
+      <mass value="0.5"/>
+      <inertia ixx="6.721e-04" ixy="0" ixz="0"
+               iyy="6.721e-04" iyz="0"
+               izz="1.3141e-03" />
+    </inertial>
+  </link>
+  <gazebo reference="blocker">
+      <material>Gazebo/DarkOrangeTransparentOverlay</material>
+  </gazebo>
+<!-- #####    END   ##### -->
+<!-- #####  A2 PART ##### -->
+<!-- #####    END   ##### -->
+<!--
   <joint name="camera_joint" type="fixed">
     <origin xyz="0.064 -0.065 0.094" rpy="0 0 0"/>
-    <parent link="base_link"/>
+    <parent link="chassis"/>
     <child link="camera_link"/>
   </joint>

Commit message: Trying LINE-MOD to recognize the can, then the B cart

File: src/amr_description/urdf/solamr.gazebo.xacro (robot description, xacro)
@@ -82,9 +82,9 @@
       <pose>0 0 0 0 0 0</pose>
       <visualize>$(arg laser_visual)</visualize>
-      <update_rate>5</update_rate>
+      <update_rate>10</update_rate>
       <ray>
         <scan>
           <horizontal>
-            <samples>300</samples>
+            <samples>725</samples>
             <resolution>1</resolution>
             <min_angle>0.0</min_angle>
@@ -93,12 +93,12 @@
         </scan>
         <range>
-          <min>0.120</min>
-          <max>3.5</max>
-          <resolution>0.015</resolution>
+          <min>0.06</min>
+          <max>4.095</max>
+          <resolution>0.1</resolution>
         </range>
         <noise>
           <type>gaussian</type>
           <mean>0.0</mean>
-          <stddev>0.0</stddev>
+          <stddev>0.01</stddev>
         </noise>
       </ray>
@@ -114,9 +114,9 @@
       <pose>0 0 0 0 0 0</pose>
       <visualize>$(arg laser_visual)</visualize>
-      <update_rate>5</update_rate>
+      <update_rate>10</update_rate>
       <ray>
         <scan>
           <horizontal>
-            <samples>300</samples>
+            <samples>725</samples>
             <resolution>1</resolution>
             <min_angle>0.0</min_angle>
@@ -125,7 +125,7 @@
         </scan>
         <range>
-          <min>0.120</min>
-          <max>3.5</max>
-          <resolution>0.015</resolution>
+          <min>0.06</min>
+          <max>4.095</max>
+          <resolution>0.01</resolution>
         </range>
         <noise>

File: src/amr_description/urdf/solamr.urdf.xacro (robot description, xacro)
@@ -73,5 +73,5 @@
         <box size="${chassis_length} ${chassis_width} ${chassis_height}"/>
       </geometry>
-      <material name="light_black"/>
+      <material name="white"/>
     </visual>
     <collision>
@@ -230,5 +230,5 @@
 -->
       </geometry>
-      <material name="light_black"/>
+      <material name="white"/>
     </visual>
     <collision>

Commit message: two solamr control in teleop.py done

File: src/amr_description/urdf/solamr.gazebo.xacro (robot description, xacro)
@@ -26,6 +26,6 @@
   </gazebo>
   <gazebo reference="wheel_left_link">
-    <mu1>20</mu1>
-    <mu2>20</mu2>
+    <mu1>10</mu1>
+    <mu2>1</mu2>
     <kp>50000.0</kp>
     <kd>10.0</kd>
@@ -36,6 +36,6 @@
   </gazebo>
   <gazebo reference="wheel_right_link">
-    <mu1>20</mu1>
-    <mu2>20</mu2>
+    <mu1>10</mu1>
+    <mu2>1</mu2>
     <kp>50000.0</kp>
     <kd>10.0</kd>

File: src/amr_description/urdf/solamr.urdf.xacro (robot description, xacro)
@@ -263,5 +263,5 @@
     <parent link="chassis"/>
     <child link="blocker"/>
-    <origin xyz="0.083 0 .18" rpy="0 1.57 0"/>
+    <origin xyz="0.077 0 .2" rpy="0 1.57 0"/>
     <axis xyz="0 0 1"/>
   </joint>
@@ -271,18 +271,15 @@
       <origin xyz=".02 0 -0.0095" rpy="0 0 0"/>
 -->
-      <origin xyz=".02 0 -0.002" rpy="0 0 0"/>
-      <geometry>
-        <mesh filename="package://amr_description/meshes/solamr/blocker.stl" scale="0.0095 0.0095 0.0095"/>
+      <origin xyz=".015 0 -0.002" rpy="0 0 0"/>
+      <geometry>
+        <mesh filename="package://amr_description/meshes/solamr/blocker.stl" scale="0.009 0.009 0.009"/>
       </geometry>
       <material name="orange"/>
     </visual>
     <collision>
-      <!--
-      <origin xyz=".02 0 -0.0095" rpy="0 0 0"/>
--->
       <max_contacts>1</max_contacts>
       <origin xyz=".02 0 -0.00" rpy="0 0 0"/>
       <geometry>
-        <mesh filename="package://amr_description/meshes/solamr/blocker.stl" scale="0.0095 0.0095 0.0095"/>
+        <mesh filename="package://amr_description/meshes/solamr/blocker.stl" scale="0.009 0.009 0.009"/>
       </geometry>
     </collision>
