Commit message: Error plotting done.

File: src/amr_description/urdf/solamr.urdf.xacro (robot description, xacro)
@@ -307,5 +307,5 @@
 <!-- Begin of camera -->
   <joint name="camera_joint" type="fixed">
-    <origin xyz="0.33 0 0.161" rpy="0 0 0"/>
+    <origin xyz="0.33 0 0.161" rpy="0 -0.35 0"/>
     <parent link="chassis"/>
     <child link="camera_link"/>

Commit message: model path fixed

File: src/amr_description/urdf/solamr.urdf.xacro (robot description, xacro)
@@ -38,5 +38,5 @@
           <origin rpy= "${PI/2} 0 0" xyz= "0 0 -0.025"/>
           <geometry>
-            <mesh filename="package://amr_description/meshes/caster.stl" scale="0.0002 0.0002 0.0002"/>
+              <mesh filename="package://amr_description/meshes/solamr/caster.stl" scale="0.0002 0.0002 0.0002"/>
           </geometry>
           <material name= "grey"/>
@@ -99,5 +99,5 @@
       <origin xyz="0 0 0" rpy="1.57 0 0"/>
       <geometry>
-        <mesh filename="package://turtlebot3_description/meshes/wheels/left_tire.stl" scale="0.001 0.001 0.001"/>
+          <mesh filename="package://amr_description/meshes/solamr/left_tire.stl" scale="0.001 0.001 0.001"/>
       </geometry>
       <material name="dark"/>
@@ -127,5 +127,5 @@
       <origin xyz="0 0 0" rpy="1.57 0 0"/>
       <geometry>
-        <mesh filename="package://turtlebot3_description/meshes/wheels/right_tire.stl" scale="0.001 0.001 0.001"/>
+          <mesh filename="package://amr_description/meshes/solamr/right_tire.stl" scale="0.001 0.001 0.001"/>
       </geometry>
       <material name="dark"/>
@@ -225,7 +225,7 @@
       <origin xyz="0.0 0 0.0" rpy="0 0 -${PI/2}"/>
       <geometry>
-        <mesh filename="package://amr_description/meshes/A2_top_H.stl" scale="0.01 0.01 0.01"/>
+        <mesh filename="package://amr_description/meshes/solamr/A2_top_H.stl" scale="0.01 0.01 0.01"/>
         <!--
-        <mesh filename="package://amr_description/meshes/A2_top_extr10mm_H.stl" scale="0.01 0.01 0.01"/>
+        <mesh filename="package://amr_description/meshes/solamr/A2_top_extr10mm_H.stl" scale="0.01 0.01 0.01"/>
 -->
       </geometry>
@@ -236,7 +236,7 @@
       <origin xyz="0.0 0 0.0" rpy="0 0 -${PI/2}"/>
       <geometry>
-        <mesh filename="package://amr_description/meshes/A2_top_H.stl" scale="0.01 0.01 0.01"/>
+        <mesh filename="package://amr_description/meshes/solamr/A2_top_H.stl" scale="0.01 0.01 0.01"/>
         <!--
-        <mesh filename="package://amr_description/meshes/A2_top_extr10mm_H.stl" scale="0.01 0.01 0.01"/>
+        <mesh filename="package://amr_description/meshes/solamr/A2_top_extr10mm_H.stl" scale="0.01 0.01 0.01"/>
 -->
       </geometry>
@@ -273,5 +273,5 @@
       <origin xyz=".02 0 -0.002" rpy="0 0 0"/>
       <geometry>
-        <mesh filename="package://amr_description/meshes/blocker.stl" scale="0.0095 0.0095 0.0095"/>
+        <mesh filename="package://amr_description/meshes/solamr/blocker.stl" scale="0.0095 0.0095 0.0095"/>
       </geometry>
       <material name="orange"/>
@@ -284,5 +284,5 @@
       <origin xyz=".02 0 -0.00" rpy="0 0 0"/>
       <geometry>
-        <mesh filename="package://amr_description/meshes/blocker.stl" scale="0.0095 0.0095 0.0095"/>
+        <mesh filename="package://amr_description/meshes/solamr/blocker.stl" scale="0.0095 0.0095 0.0095"/>
       </geometry>
     </collision>
@@ -315,5 +315,5 @@
      <origin xyz="0 0 0" rpy="1.57 0 1.57"/>
       <geometry>
-       <mesh filename="package://turtlebot3_description/meshes/sensors/r200.dae" />
+          <mesh filename="package://amr_description/meshes/sensors/r200.dae" />
       </geometry>
     </visual>

Commit message: cooperate the stl file from turtlebot

File: src/amr_description/urdf/solamr.urdf.xacro (robot description, xacro)
@@ -99,5 +99,5 @@
       <origin xyz="0 0 0" rpy="1.57 0 0"/>
       <geometry>
-        <mesh filename="package://turtlebot3_description/meshes/wheels/left_tire.stl" scale="0.001 0.001 0.001"/>
+        <mesh filename="package://amr_description/meshes/left_tire.stl" scale="0.001 0.001 0.001"/>
       </geometry>
       <material name="dark"/>
@@ -127,5 +127,5 @@
       <origin xyz="0 0 0" rpy="1.57 0 0"/>
       <geometry>
-        <mesh filename="package://turtlebot3_description/meshes/wheels/right_tire.stl" scale="0.001 0.001 0.001"/>
+          <mesh filename="package://amr_description/meshes/right_tire.stl" scale="0.001 0.001 0.001"/>
       </geometry>
       <material name="dark"/>
@@ -299,7 +299,4 @@
     </inertial>
   </link>
-  <gazebo reference="blocker">
-      <material>Gazebo/DarkOrangeTransparentOverlay</material>
-  </gazebo>
 <!-- #####    END   ##### -->
 <!-- #####  A2 PART ##### -->
@@ -315,5 +312,5 @@
      <origin xyz="0 0 0" rpy="1.57 0 1.57"/>
       <geometry>
-       <mesh filename="package://turtlebot3_description/meshes/sensors/r200.dae" />
+       <mesh filename="package://amr_description/meshes/r200.dae" />
       </geometry>
     </visual>
