Commit message: make sure it's there.....

File: src/amr_description/urdf/solamr_rod.urdf.xacro (robot description, xacro)
@@ -43,5 +43,5 @@
         </visual>
         <collision>
-          <origin rpy= "${PI/2} 0 0" xyz= "0 0 ${caster_radius + 0.0011}"/>
+          <origin rpy= "${PI/2} 0 0" xyz= "0 0 ${caster_radius + 0.001}"/>
           <geometry>
             <cylinder length="${caster_length}" radius= "${caster_radius}"/>
