Commit message: solamr and shelft connected with revolute joint

File: src/amr_description/urdf/2in1.gazebo.xacro (robot description, xacro)
@@ -9,8 +9,19 @@
     </plugin>
   </gazebo>
-  <gazebo reference="chassis">
+<!--
+  <gazebo>
+    <plugin name="joint_state_publisher" filename="libgazebo_ros_joint_state_publisher.so">
+      <robotNamespace>$(arg robotName)</robotNamespace>
+      <jointName>rear_right_wheel_joint, rear_left_wheel_joint, front_right_wheel_joint, front_left_wheel_joint, front_right_steer_joint, front_left_steer_joint, steering_joint</jointName>
+      <updateRate>100.0</updateRate>
+      <alwaysOn>true</alwaysOn>
+    </plugin>
+  </gazebo>
+-->
+<!-- FOR 2-in-1 -->
+  <gazebo reference="chassis_1">
       <material>Gazebo/CeilingTiled</material>
   </gazebo>
-  <gazebo reference="A2_top">
+  <gazebo reference="A2_top_1">
       <material>Gazebo/PointCloud</material>
       <mu1>10</mu1>
@@ -21,51 +32,32 @@
       <minDepth>0.001</minDepth>
   </gazebo>
-  <gazebo reference="blocker">
-      <material>Gazebo/OrangeTransparentOverlay</material>
-      <mu1>0</mu1>
-      <mu2>0</mu2>
-      <kp>1000000</kp>
-      <kd>10</kd>
-      <maxVel>0.</maxVel>
-      <minDepth>0.001</minDepth>
-  </gazebo>
-  <gazebo reference="wheel_left_link">
-    <mu1>10</mu1>
-    <mu2>10</mu2>
-    <kp>1000000.0</kp>
-    <kd>10.0</kd>
-    <minDepth>0.001</minDepth>
-    <maxVel>3</maxVel>
-    <fdir1>1 0 0</fdir1>
-    <material>Gazebo/FlatBlack</material>
-  </gazebo>
-  <gazebo reference="wheel_right_link">
-    <mu1>10</mu1>
-    <mu2>10</mu2>
-    <kp>1000000.0</kp>
-    <kd>10.0</kd>
-    <minDepth>0.001</minDepth>
-    <maxVel>3</maxVel>
-    <fdir1>1 0 0</fdir1>
-    <material>Gazebo/FlatBlack</material>
-  </gazebo>
-  <!--
-  <gazebo>
-    <plugin name="joint_state_publisher" filename="libgazebo_ros_joint_state_publisher.so">
-      <robotNamespace>$(arg robotName)</robotNamespace>
-      <jointName>rear_right_wheel_joint, rear_left_wheel_joint, front_right_wheel_joint, front_left_wheel_joint, front_right_steer_joint, front_left_steer_joint, steering_joint</jointName>
-      <updateRate>100.0</updateRate>
-      <alwaysOn>true</alwaysOn>
-    </plugin>
-  </gazebo>
--->
-  <gazebo>
-    <plugin name="solamr_controller" filename="libgazebo_ros_diff_drive.so">
-      <commandTopic>cmd_vel</commandTopic>
-      <odometryTopic>odom</odometryTopic>
-      <odometryFrame>odom</odometryFrame>
+  <gazebo reference="wheel_left_link_1">
+    <mu1>10</mu1>
+    <mu2>5</mu2>
+    <kp>1000000.0</kp>
+    <kd>10.0</kd>
+    <minDepth>0.001</minDepth>
+    <maxVel>3</maxVel>
+    <fdir1>1 0 0</fdir1>
+    <material>Gazebo/FlatBlack</material>
+  </gazebo>
+  <gazebo reference="wheel_right_link_1">
+    <mu1>10</mu1>
+    <mu2>5</mu2>
+    <kp>1000000.0</kp>
+    <kd>10.0</kd>
+    <minDepth>0.001</minDepth>
+    <maxVel>3</maxVel>
+    <fdir1>1 0 0</fdir1>
+    <material>Gazebo/FlatBlack</material>
+  </gazebo>
+  <gazebo>
+    <plugin name="solamr_controller_1" filename="libgazebo_ros_diff_drive.so">
+      <commandTopic>cmd_vel_1</commandTopic>
+      <odometryTopic>odom_1</odometryTopic>
+      <odometryFrame>odom_1</odometryFrame>
       <odometrySource>world</odometrySource>
       <publishOdomTF>true</publishOdomTF>
-      <robotBaseFrame>base_footprint</robotBaseFrame>
+      <robotBaseFrame>base_footprint_1</robotBaseFrame>
       <publishWheelTF>false</publishWheelTF>
       <publishTf>true</publishTf>
@@ -73,6 +65,6 @@
       <legacyMode>false</legacyMode>
       <updateRate>30</updateRate>
-      <leftJoint>wheel_left_joint</leftJoint>
-      <rightJoint>wheel_right_joint</rightJoint>
+      <leftJoint>wheel_left_joint_1</leftJoint>
+      <rightJoint>wheel_right_joint_1</rightJoint>
       <wheelSeparation>0.20</wheelSeparation>
       <wheelDiameter>0.099</wheelDiameter>
@@ -82,4 +74,59 @@
     </plugin>
   </gazebo>
+  <gazebo reference="chassis_2">
+      <material>Gazebo/CeilingTiled</material>
+  </gazebo>
+  <gazebo reference="A2_top_2">
+      <material>Gazebo/PointCloud</material>
+      <mu1>10</mu1>
+      <mu2>10</mu2>
+      <kp>1000000</kp>
+      <kd>10</kd>
+      <maxVel>0.</maxVel>
+      <minDepth>0.001</minDepth>
+  </gazebo>
+  <gazebo reference="wheel_left_link_2">
+    <mu1>10</mu1>
+    <mu2>5</mu2>
+    <kp>1000000.0</kp>
+    <kd>10.0</kd>
+    <minDepth>0.001</minDepth>
+    <maxVel>3</maxVel>
+    <fdir1>1 0 0</fdir1>
+    <material>Gazebo/FlatBlack</material>
+  </gazebo>
+  <gazebo reference="wheel_right_link_2">
+    <mu1>10</mu1>
+    <mu2>5</mu2>
+    <kp>1000000.0</kp>
+    <kd>10.0</kd>
+    <minDepth>0.001</minDepth>
+    <maxVel>3</maxVel>
+    <fdir1>1 0 0</fdir1>
+    <material>Gazebo/FlatBlack</material>
+  </gazebo>
+  <gazebo>
+    <plugin name="solamr_controller_2" filename="libgazebo_ros_diff_drive.so">
+      <commandTopic>cmd_vel_2</commandTopic>
+      <odometryTopic>odom_2</odometryTopic>
+      <odometryFrame>odom_2</odometryFrame>
+      <odometrySource>world</odometrySource>
+      <publishOdomTF>true</publishOdomTF>
+      <robotBaseFrame>base_footprint_2</robotBaseFrame>
+      <publishWheelTF>false</publishWheelTF>
+      <publishTf>true</publishTf>
+      <publishWheelJointState>true</publishWheelJointState>
+      <legacyMode>false</legacyMode>
+      <updateRate>30</updateRate>
+      <leftJoint>wheel_left_joint_2</leftJoint>
+      <rightJoint>wheel_right_joint_2</rightJoint>
+      <wheelSeparation>0.20</wheelSeparation>
+      <wheelDiameter>0.099</wheelDiameter>
+      <wheelAcceleration>10</wheelAcceleration>
+      <wheelTorque>100</wheelTorque>
+      <rosDebugLevel>na</rosDebugLevel>
+    </plugin>
+  </gazebo>
+<?ignore
   <gazebo reference="scan_front">
     <material>Gazebo/FlatBlack</material>
@@ -146,41 +193,4 @@
     </sensor>
   </gazebo>
-<!--
-  <gazebo reference="imu_link">
-    <sensor type="imu" name="imu">
-      <always_on>true</always_on>
-      <visualize>$(arg imu_visual)</visualize>
-    </sensor>
-    <material>Gazebo/Grey</material>
-  </gazebo>
-  <gazebo>
-    <plugin name="imu_plugin" filename="libgazebo_ros_imu.so">
-      <alwaysOn>true</alwaysOn>
-      <bodyName>imu_link</bodyName>
-      <frameName>imu_link</frameName>
-      <topicName>imu</topicName>
-      <serviceName>imu_service</serviceName>
-      <gaussianNoise>0.0</gaussianNoise>
-      <updateRate>200</updateRate>
-      <imu>
-        <noise>
-          <type>gaussian</type>
-          <rate>
-            <mean>0.0</mean>
-            <stddev>2e-4</stddev>
-            <bias_mean>0.0000075</bias_mean>
-            <bias_stddev>0.0000008</bias_stddev>
-          </rate>
-          <accel>
-            <mean>0.0</mean>
-            <stddev>1.7e-2</stddev>
-            <bias_mean>0.1</bias_mean>
-            <bias_stddev>0.001</bias_stddev>
-          </accel>
-        </noise>
-      </imu>
-    </plugin>
-  </gazebo>
--->
   <gazebo reference="camera_rgb_frame">
     <sensor type="depth" name="realsense_R200">
@@ -190,8 +200,4 @@
           <horizontal_fov>1.3439</horizontal_fov>
           <image>
-              <!--
-              <width>1280</width>
-              <height>720</height>
--->
               <width>640</width>
               <height>480</height>
@@ -230,3 +236,42 @@
     </sensor>
   </gazebo>
+<!--
+  <gazebo reference="imu_link">
+    <sensor type="imu" name="imu">
+      <always_on>true</always_on>
+      <visualize>$(arg imu_visual)</visualize>
+    </sensor>
+    <material>Gazebo/Grey</material>
+  </gazebo>
+  <gazebo>
+    <plugin name="imu_plugin" filename="libgazebo_ros_imu.so">
+      <alwaysOn>true</alwaysOn>
+      <bodyName>imu_link</bodyName>
+      <frameName>imu_link</frameName>
+      <topicName>imu</topicName>
+      <serviceName>imu_service</serviceName>
+      <gaussianNoise>0.0</gaussianNoise>
+      <updateRate>200</updateRate>
+      <imu>
+        <noise>
+          <type>gaussian</type>
+          <rate>
+            <mean>0.0</mean>
+            <stddev>2e-4</stddev>
+            <bias_mean>0.0000075</bias_mean>
+            <bias_stddev>0.0000008</bias_stddev>
+          </rate>
+          <accel>
+            <mean>0.0</mean>
+            <stddev>1.7e-2</stddev>
+            <bias_mean>0.1</bias_mean>
+            <bias_stddev>0.001</bias_stddev>
+          </accel>
+        </noise>
+      </imu>
+    </plugin>
+  </gazebo>
+-->
+?>
+<!-- END of  2-in-1 -->
 </robot>

File: src/amr_description/urdf/shelft_XL_rod.urdf.xacro (robot description, xacro)
@@ -5,5 +5,5 @@
 <xacro:property name="PI" value="3.14"/>
 <!-- #### body property #### -->
-<xacro:property name="body_length" value=".45"/>
+<xacro:property name="body_length" value="1.2"/>
 <xacro:property name="body_width" value=".45"/>
 <xacro:property name="body_height" value=".45"/>
@@ -13,7 +13,7 @@
 <xacro:property name="leg_mass" value="2.5"/>
 <!-- ####  rod property #### -->
-<xacro:property name="rod_radius" value="0.025"/>
-<xacro:property name="rod_length" value="0.3607"/>
-<xacro:property name="rod_mass" value="5"/>
+<xacro:property name="rod_radius" value="0.031"/>
+<xacro:property name="rod_length" value="0.3596"/>
+<xacro:property name="rod_mass" value="1.0"/>
 <!-- ####  Aruco property #### -->
 <xacro:property name="aruco_width" value="0.25"/>
@@ -59,5 +59,5 @@
       <material name= "light_black"/>
     </visual>
-    -->
+-->
     <collision>
       <origin rpy= "0 0 0" xyz= "0 0 0"/>
@@ -73,5 +73,5 @@
     <kp value="10000000.0"/>
     <kd value= "10.0"/>
-    <maxVel>3</maxVel>
+    <maxVel>0.</maxVel>
     <minDepth>0.001</minDepth>
   </gazebo>
@@ -172,5 +172,5 @@
       <origin rpy="0 0 0" xyz="0 0 0"/>
       <geometry>
-          <mesh filename="package://amr_description/meshes/shelft/only_shelft_S.stl" scale="0.01 0.01 0.01"/>
+          <mesh filename="package://amr_description/meshes/shelft/only_shelft_XL.stl" scale="0.01 0.01 0.01"/>
       </geometry>
     </visual>
@@ -196,11 +196,34 @@
   <xacro:ball_leg prefix="left" suffix="front" X1="1" Y1="1"/>
   <xacro:ball_leg prefix="left" suffix="back" X1="-1" Y1="1"/>
-<!-- #### B bottom #### -->
-  <joint name="B_bot_joint" type="fixed">
+<!-- #### B bottom 1 #### -->
+  <joint name="B_bot_1_joint" type="fixed">
     <parent link="body"/>
-    <child link="B_bot" />
-    <origin xyz="0 0 ${leg_length-0.025} " rpy="0 0 0"/>
-  </joint>
-  <link name="B_bot">
+    <child link="B_bot_1" />
+    <origin xyz="${body_length/2 - 0.22} 0 ${leg_length-0.025} " rpy="0 0 0"/>
+  </joint>
+  <link name="B_bot_1">
+    <visual>
+      <origin xyz="0.0 0 0.0" rpy="${PI} 0 ${PI/2}"/>
+      <geometry>
+        <cylinder length="${rod_length}" radius= "${rod_radius}"/>
+      </geometry>
+      <material name="light_black"/>
+    </visual>
+    <collision>
+      <max_contacts>1</max_contacts>
+      <origin xyz="0.0 0 0.0" rpy="${PI} 0 ${PI/2}"/>
+      <geometry>
+        <cylinder length="${rod_length}" radius= "${rod_radius}"/>
+      </geometry>
+    </collision>
+    <xacro:cylinder_inertia m="${rod_mass}" r="${rod_radius}" h="${rod_length}"/>
+  </link>
+<!-- #### B bottom 2 #### -->
+  <joint name="B_bot_2_joint" type="fixed">
+    <parent link="body"/>
+    <child link="B_bot_2" />
+    <origin xyz="${-body_length/2 + 0.22} 0 ${leg_length -0.025} " rpy="0 0 0"/>
+  </joint>
+  <link name="B_bot_2">
     <visual>
       <origin xyz="0.0 0 0.0" rpy="${PI} 0 ${PI/2}"/>
@@ -224,7 +247,7 @@
   <xacro:aruco prefix="north" X1="1" Y1="0" Yaw="1" aruco_id="200"/>
   <xacro:aruco prefix="south" X1="-1" Y1="0" Yaw="1" aruco_id="202"/>
-  <gazebo reference="B_bot">
-      <mu1>2</mu1>
-      <mu2>1</mu2>
+  <gazebo reference="B_bot_1">
+      <mu1>10</mu1>
+      <mu2>10</mu2>
       <kp>1000000</kp>
       <kd>10</kd>
@@ -233,3 +256,12 @@
       <material>Gazebo/Wood</material>
   </gazebo>
+  <gazebo reference="B_bot_2">
+      <mu1>10</mu1>
+      <mu2>10</mu2>
+      <kp>1000000</kp>
+      <kd>10</kd>
+      <maxVel>0.</maxVel>
+      <minDepth>0.001</minDepth>
+      <material>Gazebo/Wood</material>
+  </gazebo>
 </robot>

File: src/amr_description/urdf/solamr.urdf.xacro (robot description, xacro)
@@ -31,5 +31,5 @@
         <parent link= "chassis"/>
         <child link= "${prefix}_${suffix}_caster"/>
-        <origin xyz= "${(chassis_length/2)*X1 + (chassis_length/2-.05)*X2} ${(chassis_width/2-0.02)*Y1 + (chassis_width/2)*Y2}  0.026" rpy="0 0 0"/>
+        <origin xyz= "${(chassis_length/2)*X1 + (chassis_length/2-.05)*X2} ${(chassis_width/2-0.02)*Y1 + (chassis_width/2)*Y2}  ${caster_radius + 0.01}" rpy="0 0 0"/>
         <dynamics damping="0.0" friction="0.0"/>
       </joint>
@@ -92,5 +92,5 @@
     <parent link="chassis"/>
     <child link="wheel_left_link"/>
-    <origin xyz="0.0 ${chassis_width/2-0.05} 0.033" rpy="-1.57 0 0"/>
+    <origin xyz="0.0 ${chassis_width/2-0.05} 0.025" rpy="-1.57 0 0"/>
     <axis xyz="0 0 1"/>
   </joint>
@@ -120,5 +120,5 @@
     <parent link="chassis"/>
     <child link="wheel_right_link"/>
-    <origin xyz="0.0 -${chassis_width/2-0.05} 0.033" rpy="-1.57 0 0"/>
+    <origin xyz="0.0 -${chassis_width/2-0.05} 0.025" rpy="-1.57 0 0"/>
     <axis xyz="0 0 1"/>
   </joint>

File: src/amr_description/urdf/solamr_rod.urdf.xacro (robot description, xacro)
@@ -31,10 +31,10 @@
         <parent link= "chassis"/>
         <child link= "${prefix}_${suffix}_caster"/>
-        <origin xyz= "${(chassis_length/2)*X1 + (chassis_length/2-.05)*X2} ${(chassis_width/2-0.02)*Y1 + (chassis_width/2)*Y2}  0.026" rpy="0 0 0"/>
+        <origin xyz= "${(chassis_length/2)*X1 + (chassis_length/2-.05)*X2} ${(chassis_width/2-0.02)*Y1 + (chassis_width/2)*Y2} 0 " rpy="0 0 0"/>
         <dynamics damping="0.0" friction="0.0"/>
       </joint>
       <link name= "${prefix}_${suffix}_caster">
         <visual>
-          <origin rpy= "${PI/2} 0 0" xyz= "0 0 -0.025"/>
+          <origin rpy= "${PI/2} 0 0" xyz= "0 0 0"/>
           <geometry>
               <mesh filename="package://amr_description/meshes/solamr/caster.stl" scale="0.0002 0.0002 0.0002"/>
@@ -43,5 +43,5 @@
         </visual>
         <collision>
-          <origin rpy= "${PI/2} 0 0" xyz= "0 0 0"/>
+          <origin rpy= "${PI/2} 0 0" xyz= "0 0 ${caster_radius + 0.0011}"/>
           <geometry>
             <cylinder length="${caster_length}" radius= "${caster_radius}"/>
@@ -83,5 +83,5 @@
     <inertial>
       <origin xyz="0 0 0" rpy="0 0 0"/>
-      <mass value="15"/>
+      <mass value="50"/>
       <inertia ixx="1.15625e-01" ixy="0" ixz="0"
                iyy="1.15625e-01" iyz="0"
@@ -92,5 +92,5 @@
     <parent link="chassis"/>
     <child link="wheel_left_link"/>
-    <origin xyz="0.0 ${chassis_width/2-0.05} 0.033" rpy="-1.57 0 0"/>
+    <origin xyz="0.0 ${chassis_width/2-0.05} ${0.033*1.5}" rpy="-1.57 0 0"/>
     <axis xyz="0 0 1"/>
   </joint>
@@ -99,5 +99,5 @@
       <origin xyz="0 0 0" rpy="1.57 0 0"/>
       <geometry>
-          <mesh filename="package://amr_description/meshes/solamr/left_tire.stl" scale="0.001 0.001 0.001"/>
+          <mesh filename="package://amr_description/meshes/solamr/left_tire.stl" scale="0.0015 0.0015 0.0015"/>
       </geometry>
       <material name="dark"/>
@@ -106,5 +106,5 @@
       <origin xyz="0 0 0" rpy="0 0 0"/>
       <geometry>
-        <cylinder length="0.018" radius="0.033"/>
+          <cylinder length="0.018" radius="${0.033*1.5}"/>
       </geometry>
     </collision>
@@ -120,5 +120,5 @@
     <parent link="chassis"/>
     <child link="wheel_right_link"/>
-    <origin xyz="0.0 -${chassis_width/2-0.05} 0.033" rpy="-1.57 0 0"/>
+    <origin xyz="0.0 -${chassis_width/2-0.05} ${0.033*1.5}" rpy="-1.57 0 0"/>
     <axis xyz="0 0 1"/>
   </joint>
@@ -127,5 +127,5 @@
       <origin xyz="0 0 0" rpy="1.57 0 0"/>
       <geometry>
-          <mesh filename="package://amr_description/meshes/solamr/right_tire.stl" scale="0.001 0.001 0.001"/>
+          <mesh filename="package://amr_description/meshes/solamr/right_tire.stl" scale="0.0015 0.0015 0.0015"/>
       </geometry>
       <material name="dark"/>
@@ -134,5 +134,5 @@
       <origin xyz="0 0 0" rpy="0 0 0"/>
       <geometry>
-        <cylinder length="0.018" radius="0.033"/>
+          <cylinder length="0.018" radius="${0.033*1.5}"/>
       </geometry>
     </collision>
@@ -208,9 +208,4 @@
 <!-- #####  A1 PART ##### -->
 <!-- #####    END   ##### -->
-<gazebo>
-  <plugin name="gazebo_ros_control" filename="libgazebo_ros_control.so">
-    <robotSimType>gazebo_ros_control/DefaultRobotHWSim</robotSimType>
-  </plugin>
-</gazebo>
 <!-- #####   BEGIN  ##### -->
 <!-- #####  A2 PART ##### -->
@@ -219,13 +214,12 @@
     <parent link="chassis"/>
     <child link="A2_top" />
-    <origin xyz="0 0 0.18" rpy="0 0 0"/>
+    <origin xyz="0 0 0.1" rpy="0 0 0"/>
   </joint>
   <link name="A2_top">
     <visual>
-      <origin xyz="0.0 0 0.0" rpy="0 0 -${PI/2}"/>
-      <geometry>
-          <mesh filename="package://amr_description/meshes/solamr/A2_top_H.stl" scale="0.02 ${0.01*chassis_length/0.65} 0.01"/>
+      <origin xyz="0.0 0 0.0" rpy="0 0 0"/>
+      <geometry>
+          <mesh filename="package://amr_description/meshes/solamr/rod_A_top_100.stl" scale="0.0065 0.0065 0.0065"/>
         <!--
-        <mesh filename="package://amr_description/meshes/solamr/A2_top_extr10mm_H.stl" scale="0.01 0.01 0.01"/>
 -->
       </geometry>
@@ -234,9 +228,8 @@
     <collision>
       <max_contacts>1</max_contacts>
-      <origin xyz="0.0 0 0.0" rpy="0 0 -${PI/2}"/>
-      <geometry>
-          <mesh filename="package://amr_description/meshes/solamr/A2_top_H.stl" scale="0.02 ${0.01*chassis_length/0.65} 0.01"/>
+      <origin xyz="0.0 0 0.0" rpy="0 0 0"/>
+      <geometry>
+          <mesh filename="package://amr_description/meshes/solamr/rod_A_top_100.stl" scale="0.0065 0.0065 0.0065"/>
         <!--
-        <mesh filename="package://amr_description/meshes/solamr/A2_top_extr10mm_H.stl" scale="0.01 0.01 0.01"/>
 -->
       </geometry>
@@ -263,5 +256,5 @@
     <parent link="chassis"/>
     <child link="blocker"/>
-    <origin xyz="-0.02 0 .2" rpy="0 1.57 0"/>
+    <origin xyz="0.04 0 .1" rpy="0 1.57 0"/>
     <axis xyz="0 0 1"/>
   </joint>
