Commit message: 1. joint_state published. 2. yaw of both SOLamrs are published in /imu_*/theta

File: src/amr_description/urdf/2in1.urdf.xacro (robot description, xacro)
@@ -1,167 +1,167 @@
 <?xml version="1.0" ?>
 <robot name="$(arg robotName)" xmlns:xacro="http://ros.org/wiki/xacro">
-<!-- #### constants #### -->
-<xacro:property name="deg_to_rad" value="0.017453"/>
-<xacro:property name="PI" value="3.14"/>
-<!-- #### body property #### -->
-<xacro:property name="body_length" value="1.2"/>
-<xacro:property name="body_width" value=".45"/>
-<xacro:property name="body_height" value=".45"/>
-<!-- ####  leg property #### -->
-<xacro:property name="leg_radius" value="0.025"/>
-<xacro:property name="leg_length" value="0.32"/>
-<xacro:property name="leg_mass" value="2.5"/>
-<!-- ####  rod property #### -->
-<xacro:property name="rod_radius" value="0.031"/>
-<xacro:property name="rod_length" value="0.3596"/>
-<xacro:property name="rod_mass" value="1.0"/>
-<!-- ####  Aruco property #### -->
-<xacro:property name="aruco_width" value="0.25"/>
-<xacro:property name="aruco_length" value="0.25"/>
-<xacro:property name="aruco_height" value="0.01"/>
-<xacro:property name="aruco_z" value="1."/>
-<xacro:property name="aruco_mass" value="0.1"/>
-<xacro:property name="edge_width" value="0.1"/>
-<!-- ######################################### -->
-<!-- begin           MACRO               begin -->
-<!-- ######################################### -->
-<xacro:macro name="cylinder_inertia" params ="m r h">
-    <inertial>
-        <mass value="${m}"/>
-        <inertia ixx="${m*(3*r*r+h*h)/12}" ixy="0.0" ixz="0.0"
-                 iyy="${m*(3*r*r+h*h)/12}" iyz= "0.0"
-                 izz="${m*r*r/2}"/>
-     </inertial>
- </xacro:macro>
-<xacro:macro name="cuboid_inertia" params ="m w l h">
-    <inertial>
-        <mass value="${m}"/>
-        <inertia ixx="${m*(w*w+h*h)/12}" ixy="0.0" ixz="0.0"
-                 iyy="${m*(l*l+h*h)/12}" iyz= "0.0"
-                 izz="${m*(w*w+l*l)/12}"/>
-     </inertial>
- </xacro:macro>
-<!-- #####  leg macro  ##### -->
-<xacro:macro name="leg" params= "prefix suffix X1 Y1">
-  <joint name="${prefix}_${suffix}_leg_joint" type="fixed">
-    <parent link= "body"/>
-    <child link= "${prefix}_${suffix}_leg"/>
-    <origin xyz= "${(body_length/2)*X1} ${(body_width/2)*Y1}  ${leg_length/2}" rpy="0 0 0"/>
-    <dynamics damping="0.0" friction="0.0"/>
-  </joint>
-  <link name= "${prefix}_${suffix}_leg">
-    <!-- usefule to visualize when debugging
-    <visual>
-      <origin rpy= "0 0 0" xyz= "0 0 0"/>
-      <geometry>
-        <cylinder length="${leg_length}" radius= "${leg_radius}"/>
-      </geometry>
-      <material name= "light_black"/>
-    </visual>
--->
-    <collision>
-      <origin rpy= "0 0 0" xyz= "0 0 0"/>
-      <geometry>
-        <cylinder length="${leg_length}" radius= "${leg_radius}"/>
-      </geometry>
-    </collision>
-    <xacro:cylinder_inertia m="${leg_mass}" r="${leg_radius}" h="${leg_length}"/>
-  </link>
-  <gazebo reference ="${prefix}_${suffix}_leg">
-    <mu1 value=".005"/>
-    <mu2 value=".005"/>
-    <kp value="10000000.0"/>
-    <kd value= "10.0"/>
-    <maxVel>0.</maxVel>
-    <minDepth>0.001</minDepth>
-  </gazebo>
-</xacro:macro>
-<xacro:macro name="ball_leg" params= "prefix suffix X1 Y1">
-  <joint name="${prefix}_${suffix}_ball_leg_joint" type="fixed">
-    <parent link= "body"/>
-    <child link= "${prefix}_${suffix}_leg"/>
-    <origin xyz= "${(body_length/2)*X1} ${(body_width/2)*Y1}  ${leg_radius}" rpy="0 0 0"/>
-    <dynamics damping="0.0" friction="0.0"/>
-  </joint>
-  <link name= "${prefix}_${suffix}_leg">
-    <!-- usefule to visualize when debugging
-    <visual>
-      <origin rpy= "0 0 0" xyz= "0 0 0"/>
-      <geometry>
-        <sphere radius= "${leg_radius}"/>
-      </geometry>
-      <material name= "light_black"/>
-    </visual>
+    <!-- #### constants #### -->
+    <xacro:property name="deg_to_rad" value="0.017453"/>
+    <xacro:property name="PI" value="3.14"/>
+    <!-- #### body property #### -->
+    <xacro:property name="body_length" value="1.2"/>
+    <xacro:property name="body_width" value=".45"/>
+    <xacro:property name="body_height" value=".45"/>
+    <!-- ####  leg property #### -->
+    <xacro:property name="leg_radius" value="0.025"/>
+    <xacro:property name="leg_length" value="0.32"/>
+    <xacro:property name="leg_mass" value="2.5"/>
+    <!-- ####  rod property #### -->
+    <xacro:property name="rod_radius" value="0.031"/>
+    <xacro:property name="rod_length" value="0.3596"/>
+    <xacro:property name="rod_mass" value="1.0"/>
+    <!-- ####  Aruco property #### -->
+    <xacro:property name="aruco_width" value="0.25"/>
+    <xacro:property name="aruco_length" value="0.25"/>
+    <xacro:property name="aruco_height" value="0.01"/>
+    <xacro:property name="aruco_z" value="1."/>
+    <xacro:property name="aruco_mass" value="0.1"/>
+    <xacro:property name="edge_width" value="0.1"/>
+    <!-- ######################################### -->
+    <!-- begin           MACRO               begin -->
+    <!-- ######################################### -->
+    <xacro:macro name="cylinder_inertia" params ="m r h">
+        <inertial>
+            <mass value="${m}"/>
+            <inertia ixx="${m*(3*r*r+h*h)/12}" ixy="0.0" ixz="0.0"
+                     iyy="${m*(3*r*r+h*h)/12}" iyz= "0.0"
+                     izz="${m*r*r/2}"/>
+         </inertial>
+     </xacro:macro>
+    <xacro:macro name="cuboid_inertia" params ="m w l h">
+        <inertial>
+            <mass value="${m}"/>
+            <inertia ixx="${m*(w*w+h*h)/12}" ixy="0.0" ixz="0.0"
+                     iyy="${m*(l*l+h*h)/12}" iyz= "0.0"
+                     izz="${m*(w*w+l*l)/12}"/>
+         </inertial>
+     </xacro:macro>
+    <!-- #####  leg macro  ##### -->
+    <xacro:macro name="leg" params= "prefix suffix X1 Y1">
+      <joint name="${prefix}_${suffix}_leg_joint" type="fixed">
+        <parent link= "body"/>
+        <child link= "${prefix}_${suffix}_leg"/>
+        <origin xyz= "${(body_length/2)*X1} ${(body_width/2)*Y1}  ${leg_length/2}" rpy="0 0 0"/>
+        <dynamics damping="0.0" friction="0.0"/>
+      </joint>
+      <link name= "${prefix}_${suffix}_leg">
+        <!-- usefule to visualize when debugging
+        <visual>
+          <origin rpy= "0 0 0" xyz= "0 0 0"/>
+          <geometry>
+            <cylinder length="${leg_length}" radius= "${leg_radius}"/>
+          </geometry>
+          <material name= "light_black"/>
+        </visual>
     -->
-    <collision>
-      <origin rpy= "0 0 0" xyz= "0 0 0"/>
-      <geometry>
-        <sphere radius= "${leg_radius}"/>
-      </geometry>
-    </collision>
-    <xacro:cylinder_inertia m="${leg_mass}" r="${leg_radius}" h="${leg_length}"/>
-  </link>
-  <gazebo reference ="${prefix}_${suffix}_ball_leg">
-    <mu1 value=".0002"/>
-    <mu2 value=".0002"/>
-    <kp value="10000000.0"/>
-    <kd value= "10.0"/>
-    <maxVel>3</maxVel>
-    <minDepth>0.001</minDepth>
-  </gazebo>
-</xacro:macro>
-<!-- #####  Aruco macro  ##### -->
-    <!-- Aruco facing four directions-->
-<xacro:macro name="aruco" params= "prefix X1 Y1 Yaw aruco_id">
-  <joint name="${prefix}_joint" type="fixed">
-    <parent link= "body"/>
-    <child link= "${prefix}_aruco"/>
-    <origin xyz= "${(body_length/2)*X1} ${(body_width/2)*Y1} ${aruco_z}" rpy="${PI/2} 0 ${Yaw*PI/2}"/>
-    <dynamics damping="0.0" friction="0.0"/>
-  </joint>
-  <link name= "${prefix}_aruco">
-    <visual>
-      <origin rpy= "0 0 0" xyz= "0 0 0"/>
-      <geometry>
-          <box size="${aruco_length} ${aruco_width} ${aruco_height}"/>
-      </geometry>
-    </visual>
-    <collision>
-      <origin rpy= "0 0 0" xyz= "0 0 0"/>
-      <geometry>
-          <box size="${aruco_length} ${aruco_width} ${aruco_height}"/>
-      </geometry>
-    </collision>
-    <xacro:cuboid_inertia m="${aruco_mass}" w="${aruco_width}" l="${aruco_length}" h="${aruco_height}"/>
-  </link>
-  <gazebo reference="${prefix}_aruco">
-      <material>SOLab/aruco${aruco_id}</material>
-  </gazebo>
-    <!-- Back Board for white edges -->
-  <joint name="${prefix}_whiteboarder_joint" type="fixed">
-    <parent link= "body"/>
-    <child link= "${prefix}_aruco_whiteboarder"/>
-    <origin xyz= "${(body_length/2-aruco_height*1/3)*X1} ${(body_width/2-aruco_height*1/3)*Y1} ${aruco_z}" rpy="${PI/2} 0 ${Yaw*PI/2}"/>
-    <dynamics damping="0.0" friction="0.0"/>
-  </joint>
-  <link name= "${prefix}_aruco_whiteboarder">
-    <visual>
-      <origin rpy= "0 0 0" xyz= "0 0 0"/>
-      <geometry>
-          <box size="${aruco_length+edge_width} ${aruco_width+edge_width} ${aruco_height}"/>
-      </geometry>
-    </visual>
-    <collision>
-      <origin rpy= "0 0 0" xyz= "0 0 0"/>
-      <geometry>
-          <box size="${aruco_length+edge_width} ${aruco_width+edge_width} ${aruco_height}"/>
-      </geometry>
-    </collision>
-    <xacro:cuboid_inertia m="${aruco_mass}" w="${aruco_width+edge_width}" l="${aruco_length+edge_width}" h="${aruco_height}"/>
-  </link>
-  <gazebo reference="${prefix}_aruco_whiteboarder">
-      <material>SOLab/WhiteGlow</material>
-  </gazebo>
-</xacro:macro>
+        <collision>
+          <origin rpy= "0 0 0" xyz= "0 0 0"/>
+          <geometry>
+            <cylinder length="${leg_length}" radius= "${leg_radius}"/>
+          </geometry>
+        </collision>
+        <xacro:cylinder_inertia m="${leg_mass}" r="${leg_radius}" h="${leg_length}"/>
+      </link>
+      <gazebo reference ="${prefix}_${suffix}_leg">
+        <mu1 value=".005"/>
+        <mu2 value=".005"/>
+        <kp value="10000000.0"/>
+        <kd value= "10.0"/>
+        <maxVel>0.</maxVel>
+        <minDepth>0.001</minDepth>
+      </gazebo>
+    </xacro:macro>
+    <xacro:macro name="ball_leg" params= "prefix suffix X1 Y1">
+      <joint name="${prefix}_${suffix}_ball_leg_joint" type="fixed">
+        <parent link= "body"/>
+        <child link= "${prefix}_${suffix}_leg"/>
+        <origin xyz= "${(body_length/2)*X1} ${(body_width/2)*Y1}  ${leg_radius}" rpy="0 0 0"/>
+        <dynamics damping="0.0" friction="0.0"/>
+      </joint>
+      <link name= "${prefix}_${suffix}_leg">
+        <!-- usefule to visualize when debugging
+        <visual>
+          <origin rpy= "0 0 0" xyz= "0 0 0"/>
+          <geometry>
+            <sphere radius= "${leg_radius}"/>
+          </geometry>
+          <material name= "light_black"/>
+        </visual>
+        -->
+        <collision>
+          <origin rpy= "0 0 0" xyz= "0 0 0"/>
+          <geometry>
+            <sphere radius= "${leg_radius}"/>
+          </geometry>
+        </collision>
+        <xacro:cylinder_inertia m="${leg_mass}" r="${leg_radius}" h="${leg_length}"/>
+      </link>
+      <gazebo reference ="${prefix}_${suffix}_ball_leg">
+        <mu1 value=".0002"/>
+        <mu2 value=".0002"/>
+        <kp value="10000000.0"/>
+        <kd value= "10.0"/>
+        <maxVel>3</maxVel>
+        <minDepth>0.001</minDepth>
+      </gazebo>
+    </xacro:macro>
+    <!-- #####  Aruco macro  ##### -->
+        <!-- Aruco facing four directions-->
+    <xacro:macro name="aruco" params= "prefix X1 Y1 Yaw aruco_id">
+      <joint name="${prefix}_joint" type="fixed">
+        <parent link= "body"/>
+        <child link= "${prefix}_aruco"/>
+        <origin xyz= "${(body_length/2)*X1} ${(body_width/2)*Y1} ${aruco_z}" rpy="${PI/2} 0 ${Yaw*PI/2}"/>
+        <dynamics damping="0.0" friction="0.0"/>
+      </joint>
+      <link name= "${prefix}_aruco">
+        <visual>
+          <origin rpy= "0 0 0" xyz= "0 0 0"/>
+          <geometry>
+              <box size="${aruco_length} ${aruco_width} ${aruco_height}"/>
+          </geometry>
+        </visual>
+        <collision>
+          <origin rpy= "0 0 0" xyz= "0 0 0"/>
+          <geometry>
+              <box size="${aruco_length} ${aruco_width} ${aruco_height}"/>
+          </geometry>
+        </collision>
+        <xacro:cuboid_inertia m="${aruco_mass}" w="${aruco_width}" l="${aruco_length}" h="${aruco_height}"/>
+      </link>
+      <gazebo reference="${prefix}_aruco">
+          <material>SOLab/aruco${aruco_id}</material>
+      </gazebo>
+        <!-- Back Board for white edges -->
+      <joint name="${prefix}_whiteboarder_joint" type="fixed">
+        <parent link= "body"/>
+        <child link= "${prefix}_aruco_whiteboarder"/>
+        <origin xyz= "${(body_length/2-aruco_height*1/3)*X1} ${(body_width/2-aruco_height*1/3)*Y1} ${aruco_z}" rpy="${PI/2} 0 ${Yaw*PI/2}"/>
+        <dynamics damping="0.0" friction="0.0"/>
+      </joint>
+      <link name= "${prefix}_aruco_whiteboarder">
+        <visual>
+          <origin rpy= "0 0 0" xyz= "0 0 0"/>
+          <geometry>
+              <box size="${aruco_length+edge_width} ${aruco_width+edge_width} ${aruco_height}"/>
+          </geometry>
+        </visual>
+        <collision>
+          <origin rpy= "0 0 0" xyz= "0 0 0"/>
+          <geometry>
+              <box size="${aruco_length+edge_width} ${aruco_width+edge_width} ${aruco_height}"/>
+          </geometry>
+        </collision>
+        <xacro:cuboid_inertia m="${aruco_mass}" w="${aruco_width+edge_width}" l="${aruco_length+edge_width}" h="${aruco_height}"/>
+      </link>
+      <gazebo reference="${prefix}_aruco_whiteboarder">
+          <material>SOLab/WhiteGlow</material>
+      </gazebo>
+    </xacro:macro>
 <!-- ##################################### -->
 <!-- end           MACRO               end -->
@@ -340,4 +340,16 @@
     <axis xyz="0 0 1"/>
   </joint>
+<!--
+  <transmission name="solamr_1_tran" type="SimpleTransmission">
+    <type>transmission_interface/SimpleTransmission</type>
+    <joint name="base_joint_1">
+      <hardwareInterface>PositionJointInterface</hardwareInterface>
+    </joint>
+    <actuator name="solamr_1_tran_motor">
+      <hardwareInterface>PositionJointInterface</hardwareInterface>
+      <mechanicalReduction>1</mechanicalReduction>
+    </actuator>
+  </transmission>
+-->
   <link name="chassis_1">
     <visual>
@@ -453,8 +465,8 @@
   <joint name="scan_joint_12" type="fixed">
     <parent link="chassis_1"/>
-    <child link="scan_rear_1"/>
+    <child link="scan_rear_12"/>
     <origin xyz="-${chassis_length/2-0.03} -${chassis_width/2-0.03} 0.16" rpy="0 0 ${PI/2}"/>
   </joint>
-  <link name="scan_rear_1">
+  <link name="scan_rear_12">
     <visual>
       <origin xyz="0 0 -.06" rpy="${PI/2} 0 0"/>
@@ -494,6 +506,4 @@
       <geometry>
           <mesh filename="package://amr_description/meshes/solamr/rod_A_top_100.stl" scale="0.0065 0.0065 0.0065"/>
-        <!--
--->
       </geometry>
       <material name="white"/>
@@ -504,6 +514,4 @@
       <geometry>
           <mesh filename="package://amr_description/meshes/solamr/rod_A_top_100.stl" scale="0.0065 0.0065 0.0065"/>
-        <!--
--->
       </geometry>
     </collision>
@@ -610,4 +618,23 @@
     <axis xyz="0 0 1"/>
   </joint>
+<!--
+  <transmission name="solamr_2_tran" type="SimpleTransmission">
+    <type>transmission_interface/SimpleTransmission</type>
+    <joint name="base_joint_2">
+      <hardwareInterface>PositionJointInterface</hardwareInterface>
+    </joint>
+    <actuator name="solamr_2_tran_motor">
+      <hardwareInterface>PositionJointInterface</hardwareInterface>
+      <mechanicalReduction>1</mechanicalReduction>
+    </actuator>
+  </transmission>
+-->
+<!--
+  <joint name="base_joint_2" type="fixed">
+    <parent link="body"/>
+    <child link="chassis_2" />
+    <origin xyz="${-body_length/2 + 0.22} 0 -0.01" rpy="0 0 0"/>
+  </joint>
+-->
   <link name="chassis_2">
     <visual>
@@ -723,8 +750,8 @@
   <joint name="scan_joint_22" type="fixed">
     <parent link="chassis_2"/>
-    <child link="scan_rear_2"/>
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
File: src/amr_description/urdf/solamr.urdf.xacro (robot description, xacro)
@@ -208,4 +208,5 @@
 <!-- #####  A1 PART ##### -->
 <!-- #####    END   ##### -->
+<!--
 <gazebo>
   <plugin name="gazebo_ros_control" filename="libgazebo_ros_control.so">
@@ -213,4 +214,5 @@
   </plugin>
 </gazebo>
+-->
 <!-- #####   BEGIN  ##### -->
 <!-- #####  A2 PART ##### -->
