Commit message: add linked_diff_drive

File: src/amr_description/urdf/2in1.gazebo.xacro (robot description, xacro)
@@ -3,5 +3,5 @@
   <xacro:arg name="laser_visual"  default="false"/>
   <xacro:arg name="camera_visual" default="false"/>
-  <xacro:arg name="imu_visual"    default="false"/>
+  <xacro:arg name="imu_visual"    default="true"/>
   <gazebo>
     <plugin name="gazebo_ros_control" filename="libgazebo_ros_control.so">
@@ -11,7 +11,4 @@
   </gazebo>
 <!-- FOR 2-in-1 -->
-  <gazebo reference="chassis_1">
-      <material>Gazebo/CeilingTiled</material>
-  </gazebo>
   <gazebo reference="A2_top_1">
       <material>Gazebo/PointCloud</material>
@@ -83,10 +80,10 @@
       <odometryTopic>odom_1</odometryTopic>
       <odometryFrame>odom_1</odometryFrame>
-      <odometrySource>world</odometrySource>
-      <publishOdomTF>false</publishOdomTF>
+      <odometrySource>map</odometrySource>
+      <publishOdomTF>true</publishOdomTF>
       <robotBaseFrame>chassis_1</robotBaseFrame>
       <publishWheelTF>false</publishWheelTF>
       <publishTf>true</publishTf>
-      <publishWheelJointState>false</publishWheelJointState>
+      <publishWheelJointState>true</publishWheelJointState>
       <legacyMode>false</legacyMode>
       <updateRate>30</updateRate>
@@ -99,7 +96,4 @@
       <rosDebugLevel>na</rosDebugLevel>
     </plugin>
-  </gazebo>
-  <gazebo reference="chassis_2">
-      <material>Gazebo/CeilingTiled</material>
   </gazebo>
   <gazebo reference="A2_top_2">
@@ -172,10 +166,10 @@
       <odometryTopic>odom_2</odometryTopic>
       <odometryFrame>odom_2</odometryFrame>
-      <odometrySource>world</odometrySource>
+      <odometrySource>map</odometrySource>
       <publishOdomTF>false</publishOdomTF>
       <robotBaseFrame>chassis_2</robotBaseFrame>
-      <publishWheelTF>false</publishWheelTF>
+      <publishWheelTF>true</publishWheelTF>
       <publishTf>true</publishTf>
-      <publishWheelJointState>false</publishWheelJointState>
+      <publishWheelJointState>true</publishWheelJointState>
       <legacyMode>false</legacyMode>
       <updateRate>30</updateRate>
@@ -189,4 +183,132 @@
     </plugin>
   </gazebo>
+  <gazebo reference="scan_front_1">
+    <material>Gazebo/FlatBlack</material>
+    <sensor type="ray" name="scan_front_1">
+      <pose>0 0 0 0 0 0</pose>
+      <visualize>$(arg laser_visual)</visualize>
+      <update_rate>10</update_rate>
+      <ray>
+        <scan>
+          <horizontal>
+            <samples>725</samples>
+            <resolution>1</resolution>
+            <min_angle>0.0</min_angle>
+            <max_angle>4.712</max_angle>
+          </horizontal>
+        </scan>
+        <range>
+          <min>0.06</min>
+          <max>4.095</max>
+          <resolution>0.1</resolution>
+        </range>
+        <noise>
+          <type>gaussian</type>
+          <mean>0.0</mean>
+          <stddev>0.01</stddev>
+        </noise>
+      </ray>
+      <plugin name="gazebo_ros_lds_lfcd_controller" filename="libgazebo_ros_laser.so">
+        <topicName>scan_front_1</topicName>
+        <frameName>scan_front_1</frameName>
+      </plugin>
+    </sensor>
+  </gazebo>
+  <gazebo reference="scan_rear_1">
+    <material>Gazebo/Blue</material>
+    <sensor type="ray" name="scan_rear_1">
+      <pose>0 0 0 0 0 0</pose>
+      <visualize>$(arg laser_visual)</visualize>
+      <update_rate>10</update_rate>
+      <ray>
+        <scan>
+          <horizontal>
+            <samples>725</samples>
+            <resolution>1</resolution>
+            <min_angle>0.0</min_angle>
+            <max_angle>4.712</max_angle>
+          </horizontal>
+        </scan>
+        <range>
+          <min>0.06</min>
+          <max>4.095</max>
+          <resolution>0.01</resolution>
+        </range>
+        <noise>
+          <type>gaussian</type>
+          <mean>0.0</mean>
+          <stddev>0.01</stddev>
+        </noise>
+      </ray>
+      <plugin name="gazebo_ros_lds_lfcd_controller" filename="libgazebo_ros_laser.so">
+        <topicName>scan_rear_1</topicName>
+        <frameName>scan_rear_1</frameName>
+      </plugin>
+    </sensor>
+  </gazebo>
+  <gazebo reference="scan_front_2">
+    <material>Gazebo/FlatBlack</material>
+    <sensor type="ray" name="scan_front_2">
+      <pose>0 0 0 0 0 0</pose>
+      <visualize>$(arg laser_visual)</visualize>
+      <update_rate>10</update_rate>
+      <ray>
+        <scan>
+          <horizontal>
+            <samples>725</samples>
+            <resolution>1</resolution>
+            <min_angle>0.0</min_angle>
+            <max_angle>4.712</max_angle>
+          </horizontal>
+        </scan>
+        <range>
+          <min>0.06</min>
+          <max>4.095</max>
+          <resolution>0.1</resolution>
+        </range>
+        <noise>
+          <type>gaussian</type>
+          <mean>0.0</mean>
+          <stddev>0.01</stddev>
+        </noise>
+      </ray>
+      <plugin name="gazebo_ros_lds_lfcd_controller" filename="libgazebo_ros_laser.so">
+        <topicName>scan_front_2</topicName>
+        <frameName>scan_front_2</frameName>
+      </plugin>
+    </sensor>
+  </gazebo>
+  <gazebo reference="scan_rear_2">
+    <material>Gazebo/Blue</material>
+    <sensor type="ray" name="scan_rear_2">
+      <pose>0 0 0 0 0 0</pose>
+      <visualize>$(arg laser_visual)</visualize>
+      <update_rate>10</update_rate>
+      <ray>
+        <scan>
+          <horizontal>
+            <samples>725</samples>
+            <resolution>1</resolution>
+            <min_angle>0.0</min_angle>
+            <max_angle>4.712</max_angle>
+          </horizontal>
+        </scan>
+        <range>
+          <min>0.06</min>
+          <max>4.095</max>
+          <resolution>0.01</resolution>
+        </range>
+        <noise>
+          <type>gaussian</type>
+          <mean>0.0</mean>
+          <stddev>0.01</stddev>
+        </noise>
+      </ray>
+      <plugin name="gazebo_ros_lds_lfcd_controller" filename="libgazebo_ros_laser.so">
+        <topicName>scan_rear_2</topicName>
+        <frameName>scan_rear_2</frameName>
+      </plugin>
+    </sensor>
+  </gazebo>
 <!-- END of  2-in-1 -->
 </robot>

File: src/amr_description/urdf/2in1.urdf.xacro (robot description, xacro)
@@ -167,4 +167,10 @@
 <!-- end           MACRO               end -->
 <!-- ##################################### -->
+  <link name="base_footprint"/>
+  <joint name="base_joint" type="fixed">
+    <parent link="base_footprint"/>
+    <child link="body" />
+    <origin xyz="0 0 0.0" rpy="0 0 0"/>
+  </joint>
   <!-- body-->
   <link name="body">
@@ -176,8 +182,14 @@
     </visual>
     <collision>
+      <origin rpy="0 0 0" xyz="0 0 0.1"/>
+      <geometry>
+          <mesh filename="package://amr_description/meshes/shelft/only_shelft_XL.stl" scale="0.01 0.01 0.01"/>
+      </geometry>
+<!--
        <origin rpy="0 0 0" xyz="0 0 ${leg_length + body_height/2}"/>
        <geometry>
         <box size="${body_length} ${body_width} ${body_height}"/>
        </geometry>
+-->
      </collision>
      <inertial>
@@ -335,7 +347,7 @@
 <!-- #####   BEGIN  ##### -->
   <joint name="base_joint_1" type="continuous">
-    <parent link="body"/>
+    <parent link="B_bot_1"/>
     <child link="chassis_1" />
-    <origin xyz="${body_length/2 - 0.22} 0 -0.01" rpy="0 0 0"/>
+    <origin xyz="0 0 ${-leg_length+0.025-0.01}" rpy="0 0 0"/>
     <axis xyz="0 0 1"/>
   </joint>
@@ -438,8 +450,8 @@
   <joint name="scan_joint_11" type="fixed">
     <parent link="chassis_1"/>
-    <child link="scan_front_11"/>
+    <child link="scan_front_1"/>
     <origin xyz="${chassis_length/2-0.03} ${chassis_width/2-0.03} 0.16" rpy="0 0 -${PI/2}"/>
   </joint>
-  <link name="scan_front_11">
+  <link name="scan_front_1">
     <visual>
       <origin xyz="0 0 -.06" rpy="${PI/2} 0 0"/>
@@ -465,8 +477,8 @@
   <joint name="scan_joint_12" type="fixed">
     <parent link="chassis_1"/>
-    <child link="scan_rear_12"/>
+    <child link="scan_rear_1"/>
     <origin xyz="-${chassis_length/2-0.03} -${chassis_width/2-0.03} 0.16" rpy="0 0 ${PI/2}"/>
   </joint>
-  <link name="scan_rear_12">
+  <link name="scan_rear_1">
     <visual>
       <origin xyz="0 0 -.06" rpy="${PI/2} 0 0"/>
@@ -723,8 +735,8 @@
   <joint name="scan_joint_21" type="fixed">
     <parent link="chassis_2"/>
-    <child link="scan_front_21"/>
+    <child link="scan_front_2"/>
     <origin xyz="${chassis_length/2-0.03} ${chassis_width/2-0.03} 0.16" rpy="0 0 -${PI/2}"/>
   </joint>
-  <link name="scan_front_21">
+  <link name="scan_front_2">
     <visual>
       <origin xyz="0 0 -.06" rpy="${PI/2} 0 0"/>
@@ -750,8 +762,8 @@
   <joint name="scan_joint_22" type="fixed">
     <parent link="chassis_2"/>
-    <child link="scan_rear_22"/>
+    <child link="scan_rear_2"/>
     <origin xyz="-${chassis_length/2-0.03} -${chassis_width/2-0.03} 0.16" rpy="0 0 ${PI/2}"/>
   </joint>
-  <link name="scan_rear_22">
+  <link name="scan_rear_2">
     <visual>
       <origin xyz="0 0 -.06" rpy="${PI/2} 0 0"/>

File: src/amr_description/urdf/solamr.gazebo.xacro (robot description, xacro)
@@ -72,5 +72,5 @@
       <publishWheelJointState>true</publishWheelJointState>
       <legacyMode>false</legacyMode>
-      <updateRate>30</updateRate>
+      <updateRate>20</updateRate>
       <leftJoint>wheel_left_joint</leftJoint>
       <rightJoint>wheel_right_joint</rightJoint>
